File: Dashboard/Dash2/Dash2/Dash2.kicad_pcb (KiCad board)
At the start: 2 copper layers, 110 x 110 mm, 164 parts, among them J101 Left_Signal, J102 Right_Signal, J103 Brake Light, J104 Headlight, J105 Backup, J106 BPS_PWR, J107 SWD, J108 Motor-C, J109 Motor-P, J110 Array-C, J111 Array-P, J112 Conn_01x03_Female, J113 Conn_01x03_Female, J114 JTAG, J115 Gecko_Cable, J201 CAN_OUT, J202 CAN_IN, J301 CarPowerConnector, J501 USB_B_Micro, SW101 CRUISE_SET, SW102 CRUISE, SW103 HAZARD, SW104 HEADLIGHT_SW, SW105 F/R_SW, SW106 BACKUP_SW, SW107 SW_Rotary2x6, SW108 TURN_SIGNAL_SW, SW109 KILL_SW, SW110 RESET, U101 EL3H7, U102 EL3H7, U103 EL3H7, U104 EL3H7, U105 EL3H7, U106 EL3H7, U107 STM32F413ZHTx, U108 EL3H7, U109 EL3H7, U110 EL3H7, U111 EL3H7, U201 ADM3055E, U202 CDSOT23-T24CAN, U301 RI3-1205S, U302 NCP1117-3.3_SOT223, U501 CP2102N-A01-GQFN24, Y101 Crystal, Y102 Crystal

Commit message: Add complete layout of the board
Parts:
- removed J107: SWD, Connector_PinHeader_2.54mm:PinHeader_1x04_P2.54mm_Vertical
- C110, C111: value C_Small -> 2.2uF
- C119, C122, C123, C124, R101, R102, R103, R107, R108, R114, R115: moved to B.Cu
- C126: value 0.1u -> 0.1uF
- C127: value 0.1u -> 0.1uF; moved to F.Cu
- L101, L102, L103, L104: footprint Diode_SMD:D_0805_2012Metric -> Inductor_SMD:L_0805_2012Metric
- R116: value 10K -> 10k
- R126: moved to F.Cu
- Y102: footprint Crystal:Crystal_SMD_TXC_7A-2Pin_5x3.2mm -> Crystal:Crystal_SMD_TXC_9HT11-2Pin_2.0x1.2mm
- moved J114 239.2 mm to (170.2, 77.7), turned to 225 degrees
- moved TP101 198.0 mm to (189.7, 157.5), turned to 180 degrees
- moved R105 166.5 mm to (179.1, 105.9), turned to 225 degrees
- moved R104 155.6 mm to (172.4, 106.3), turned to 225 degrees
- moved R114 154.4 mm to (147.3, 120.7), turned to 270 degrees
- moved C119 150.6 mm to (152.3, 74.5), turned to 45 degrees
- moved R115 148.7 mm to (148.0, 134.4), turned to 180 degrees
- moved R102 145.8 mm to (129.8, 144.4), turned to 270 degrees
- moved R107 144.6 mm to (122.9, 155.6), turned to 270 degrees
- moved R101 143.9 mm to (127.5, 148.2), turned to 90 degrees
- moved R108 142.0 mm to (110.7, 155.6), turned to 270 degrees
- moved R103 135.7 mm to (129.8, 136.8), turned to 270 degrees
- moved C123 129.6 mm to (155.3, 91.1), turned to 315 degrees
- moved C124 126.9 mm to (141.8, 71.7), turned to 135 degrees
- moved C122 119.4 mm to (147.7, 69.9), turned to 45 degrees
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Connections:
- D103 pad 1: /PB9 -> /PA2
- R104 pad 2: /PG9 -> /PB14
- R105 pad 2: /PG14 -> /PB15
- R110 pad 2: /PB9 -> /PA2
- R117 pad 2: /PD15 -> /PB5
- R118 pad 2: /PF12 -> /PB4
- R119 pad 2: /PA7 -> /PB7
- R120 pad 2: /PD14 -> /PB6
- R121 pad 2: /PD15 -> /PB5
- R122 pad 2: /PF12 -> /PB4
- R123 pad 2: /PA7 -> /PB7
- R124 pad 2: /PD14 -> /PB6
- U101 pad 4: /PG9 -> /PB14
- U102 pad 4: /PG14 -> /PB15
- U107 pad 124: /PG9 -> (no net)
- U107 pad 129: /PG14 -> (no net)
- U107 pad 134: (no net) -> /PB4
- U107 pad 135: (no net) -> /PB5
- U107 pad 136: (no net) -> /PB6
- U107 pad 137: (no net) -> /PB7
- U107 pad 140: /PB9 -> (no net)
- U107 pad 36: (no net) -> /PA2
- U107 pad 43: /PA7 -> (no net)
- U107 pad 50: /PF12 -> (no net)
- U107 pad 75: (no net) -> /PB14
- U107 pad 76: (no net) -> /PB15
- U107 pad 85: /PD14 -> (no net)
- U107 pad 86: /PD15 -> (no net)
Routing:
- net +3V3: track 0.00 -> 503.4 mm, vias 0 -> 16
- net +12V: track 0.00 -> 206.9 mm
- net /PB4: track 0.00 -> 102.1 mm, vias 0 -> 6
- net +5V: track 0.00 -> 96.7 mm, vias 0 -> 4
- net /PB8: track 0.00 -> 94.7 mm, vias 0 -> 8
- net /PB7: track 0.00 -> 86.6 mm, vias 0 -> 4
- net /PB6: track 0.00 -> 82.6 mm, vias 0 -> 4
- net /PF15: track 0.00 -> 80.8 mm, vias 0 -> 4
- net /PB5: track 0.00 -> 77.6 mm, vias 0 -> 6
- net /PE13: track 0.00 -> 74.7 mm, vias 0 -> 4
- net /PA5: track 0.00 -> 66.9 mm, vias 0 -> 4
- net Net-(J115-Pad16): track 0.00 -> 65.7 mm, vias 0 -> 6
- net Net-(J115-Pad17): track 0.00 -> 65.0 mm, vias 0 -> 6
- net /BPS_PWR: track 0.00 -> 64.7 mm
- net /PF14: track 0.00 -> 62.6 mm, vias 0 -> 2
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- added copper zone on B.Cu, net GND
- added copper zone on F.Cu, net GND
- added copper zone on B.Cu, net GNDPWR
- added copper zone on F.Cu, net GNDPWR
Other:
- net class Default: via_dia 0.8 -> 0.6; via_drill 0.4 -> 0.3
- board text added: "12V"
- board text added: "3V3"
- board text added: "A-Contact"
- board text added: "A-Precharge"
- board text added: "Array Precharge LED"
- board text added: "BPS Power"
- board text added: "BPS Power LED"
- board text added: "Backup"
- board text added: "Backup Switch"
- board text added: "BeVolt Dashboard V2 Designed by Chase Block Based on a design by Armin and Artin Taher UTSVT 2020"
- board text added: "Brake Light"
- board text added: "Brake-Pot"
- board text added: "CLK"
- board text added: "Cruise Enable"
- board text added: "Cruise Set"
- board text added: "Forward/Reverse"
- board text added: "GND"
- board text added: "Hazard Switch"
- board text added: "Headlight"
- board text added: "Headlight Switch"
- board text added: "JTDI"
- board text added: "JTDO"
- board text added: "Kill Switch"
- board text added: "Kill switch LED"
- board text added: "Left Light"
- board text added: "M-Contact"
- board text added: "M-Precharge"
- board text added: "Motor Contactor LED"
- board text added: "Motor Precharge LED"
- board text added: "Regen-Pot"
- board text added: "Right Light"
- board text added: "SWDIO"
- board text added: "Turn Signal"

Commit message: Add LED board and timing circuitry. The LED board is not yet integrated with the Dash.
Parts:
- removed D501: SP0503BAHT, Package_TO_SOT_SMD:SOT-143
- removed J115: Gecko_Cable, utsvt_conn:ribbon_cable_right_2x10
- added C401: 4.7uF, Capacitor_SMD:C_0805_2012Metric, F.Cu at (67.8, 58.3)
- added C402: 0.1uF, Capacitor_SMD:C_0805_2012Metric, F.Cu at (72.2, 58.3)
- added C503: 0.1uF, Capacitor_SMD:C_0805_2012Metric, F.Cu at (218.2, 96.9)
- added C504: 0.01uF, Capacitor_SMD:C_0805_2012Metric, F.Cu at (222.6, 93.9)
- added C505: 0.22uF, Capacitor_SMD:C_0805_2012Metric, F.Cu at (218.2, 99.8)
- added C506: 10uF, Capacitor_SMD:C_0805_2012Metric, F.Cu at (222.6, 96.9)
- added C507: 0.1uF, Capacitor_SMD:C_0805_2012Metric, F.Cu at (210.8, 110.5)
- added C508: 0.01uF, Capacitor_SMD:C_0805_2012Metric, F.Cu at (195.7, 110.5)
- added D401: SP0503BAHT, Package_TO_SOT_SMD:SOT-143, F.Cu at (78.0, 58.2)
- added J107: Gecko_Cable, utsvt_conn:ribbon_cable_right_2x10, F.Cu at (-70.9, 83.6)
- added J401: USB_B_Micro, Connector_USB:USB_Micro-B_Molex-105017-0001, F.Cu at (70.5, 52.7)
- added J502: CAN_OUT, utsvt_conn:Molex_MicroFit3.0_1x4xP3.00mm_PolarizingPeg_Vertical, F.Cu at (231.6, 78.5)
- added JP501: Termination Resistors, Connector_PinHeader_2.54mm:PinHeader_1x02_P2.54mm_Vertical, F.Cu at (216.9, 87.1)
- added L501: 2kH, Inductor_SMD:L_0805_2012Metric, F.Cu at (210.8, 107.5)
- added L502: 2kH, Inductor_SMD:L_0805_2012Metric, F.Cu at (206.4, 110.5)
- added R401: 22.1k, Resistor_SMD:R_0805_2012Metric, F.Cu at (82.8, 57.4)
- added R402: 47.5k, Resistor_SMD:R_0805_2012Metric, F.Cu at (83.9, 54.1)
- added R403: 1k, Resistor_SMD:R_0805_2012Metric, F.Cu at (83.9, 51.2)
- added TP501: CAN_H, TestPoint:TestPoint_Keystone_5005-5009_Compact, F.Cu at (196.7, 106.5)
- added TP502: CAN_L, TestPoint:TestPoint_Keystone_5005-5009_Compact, F.Cu at (191.6, 106.5)
- added U401: CP2102N-A01-GQFN24, Package_DFN_QFN:QFN-24-1EP_4x4mm_P0.5mm_EP2.6x2.6mm, F.Cu at (78.6, 52.8)
- added U502: CDSOT23-T24CAN, Package_TO_SOT_SMD:SOT-23W, F.Cu at (220.5, 73.2)
- C105, C106, C109, C110, C111, C112, C113, C114, C116, C118, C119, C122, C123, C124, C125, C126, C201, C202, C302, C303, C304, C502, J101, J102, J103, J104, J105, J106, J113, J301, R101, R102, R103, R106, R107, R108, R113, R114, R115, R116, R125, R201, U201: moved to F.Cu
- C501: value 4.7uF -> 10uF; moved to F.Cu
- J108: value Motor-C -> JTAG; footprint utsvt_conn:Molex_MicroFit3.0_1x2xP3.00mm_PolarizingPeg_Vertical -> Connector_PinHeader_2.54mm:PinHeader_1x06_P2.54mm_Vertical; moved to F.Cu
- J109: value Motor-P -> Motor-C; moved to F.Cu
- J110: value Array-C -> Motor-P; moved to F.Cu
- J111: value Array-P -> Array-C; moved to F.Cu
- J112: value Conn_01x03_Female -> Array-P; footprint utsvt_conn:Molex_MicroFit3.0_1x3xP3.00mm_PolarizingPeg_Vertical -> utsvt_conn:Molex_MicroFit3.0_1x2xP3.00mm_PolarizingPeg_Vertical; moved to F.Cu
- J114: value JTAG -> Conn_01x03_Female; footprint Connector_PinHeader_2.54mm:PinHeader_1x06_P2.54mm_Vertical -> utsvt_conn:Molex_MicroFit3.0_1x3xP3.00mm_PolarizingPeg_Vertical
- J201: value CAN_OUT -> CAN_IN; moved to F.Cu
- J202: value CAN_IN -> CAN_OUT; moved to F.Cu
- J501: value USB_B_Micro -> CAN_IN; footprint Connector_USB:USB_Micro-B_Molex-105017-0001 -> utsvt_conn:Molex_MicroFit3.0_1x4xP3.00mm_PolarizingPeg_Vertical
- R501: value 22.1k -> 0
- R502: value 47.5k -> 60
- R503: value 1k -> 60
- U501: value CP2102N-A01-GQFN24 -> ADM3055E; footprint Package_DFN_QFN:QFN-24-1EP_4x4mm_P0.5mm_EP2.6x2.6mm -> utsvt_ics:SOIC-20W_7.5x15.4mm_Pitch1.27mm
- moved JP201 260.5 mm to (-74.2, 122.1), turned to 0 degrees
- moved TP202 256.6 mm to (-69.4, 122.3), turned to 0 degrees
- moved TP201 256.4 mm to (-64.3, 122.3), turned to 0 degrees
- moved R203 255.9 mm to (-69.7, 126.3), turned to 0 degrees
- moved J201 255.7 mm to (-71.5, 116.1), turned to 0 degrees
- moved R202 249.0 mm to (-65.3, 126.3), turned to 0 degrees
- moved J202 248.0 mm to (-71.5, 108.8), turned to 0 degrees
- moved SW107 246.1 mm to (-53.2, 47.3)
- moved U202 241.3 mm to (-59.3, 124.1), turned to 0 degrees
- moved U108 239.1 mm to (-71.8, 99.5)
- moved C205 225.5 mm to (-54.7, 126.2), turned to 0 degrees
- moved L201 223.4 mm to (-50.3, 126.2), turned to 0 degrees
- moved C206 221.8 mm to (-50.3, 123.3), turned to 0 degrees
- moved U201 218.9 mm to (-51.2, 113.5)
- moved C207 217.4 mm to (-42.9, 115.6), turned to 0 degrees
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Connections:
- net /PA2 renamed /R_LGHT
- net /PA5 renamed /L_LGHT
- net /PA6 renamed /BK_LGHT
- net /PB14 renamed /IG1
- net /PB15 renamed /IG2
- net /PB4 renamed /M_PRCHG
- net /PB5 renamed /M_CNCTR
- net /PB6 renamed /A_PRCHG
- net /PB7 renamed /A_CNCTR
- net /PB8 renamed /FR_SW
- net /PE13 renamed /RIGHT_SW
- net /PE9 renamed /HZD_SW
- net /PF13 renamed /CRUZ_EN
- net /PF14 renamed /CRUZ_ST
- net /PF15 renamed /LEFT_SW
- C501 pad 1: +3V3 -> +5V
- C502 pad 1: +3V3 -> +5V
- J108 pad 1: Net-(J108-Pad1) -> /SWDIO
- J108 pad 2: Net-(J108-Pad2) -> /JTDI
- J112 pad 1: +3V3 -> Net-(J112-Pad1)
- J114 pad 1: /SWDIO -> +3V3
- J114 pad 2: /JTDI -> Net-(J114-Pad2)
- J114 pad 3: /JTDO -> GND
- J501 pad 1: Net-(D501-Pad2) -> Net-(C506-Pad1)
- J501 pad 2: Net-(D501-Pad3) -> Net-(C506-Pad2)
- J501 pad 3: Net-(D501-Pad4) -> /MotorCAN/CAN_H
- J501 pad 4: (no net) -> /MotorCAN/CAN_L
- R127 pad 1: Net-(J112-Pad2) -> Net-(J113-Pad2)
- R128 pad 1: Net-(J113-Pad2) -> Net-(J114-Pad2)
- R501 pad 1: Net-(R501-Pad1) -> /MotorCAN/RSlope
- R501 pad 2: Net-(D501-Pad2) -> Net-(C506-Pad2)
- R502 pad 1: Net-(R501-Pad1) -> /MotorCAN/TERM_H
- R502 pad 2: GND -> /MotorCAN/CAN_H
- R503 pad 1: +3V3 -> /MotorCAN/TERM_L
- R503 pad 2: Net-(R503-Pad2) -> /MotorCAN/CAN_L
- U107 pad 73: (no net) -> /MotorCAN/CAN_RX
- U107 pad 74: (no net) -> /MotorCAN/CAN_TX
- U108 pad 3: Net-(J108-Pad2) -> Net-(J109-Pad2)
- U108 pad 4: Net-(J108-Pad1) -> Net-(J109-Pad1)
- U109 pad 3: Net-(J109-Pad2) -> Net-(J110-Pad2)
- U109 pad 4: Net-(J109-Pad1) -> Net-(J110-Pad1)
- U110 pad 3: Net-(J110-Pad2) -> Net-(J111-Pad2)
- U110 pad 4: Net-(J110-Pad1) -> Net-(J111-Pad1)
- U111 pad 3: Net-(J111-Pad2) -> Net-(J112-Pad2)
- U111 pad 4: Net-(J111-Pad1) -> Net-(J112-Pad1)
- U501 pad 1: (no net) -> GND
- U501 pad 10: (no net) -> GND
- U501 pad 11: (no net) -> Net-(C506-Pad2)
- U501 pad 12: (no net) -> /MotorCAN/RSlope
- U501 pad 13: (no net) -> /MotorCAN/CAN_L
- U501 pad 14: (no net) -> /MotorCAN/CAN_H
- U501 pad 15: (no net) -> Net-(C506-Pad2)
- U501 pad 16: (no net) -> Net-(C506-Pad1)
- U501 pad 18: (no net) -> Net-(C505-Pad2)
- U501 pad 19: (no net) -> Net-(C505-Pad1)
- U501 pad 20: /USB/UART_RX -> Net-(C505-Pad2)
- U501 pad 3: Net-(D501-Pad4) -> +5V
- U501 pad 4: Net-(D501-Pad3) -> +3V3
- U501 pad 5: +3V3 -> /MotorCAN/CAN_RX
- U501 pad 6: +3V3 -> (no net)
- U501 pad 7: +3V3 -> /MotorCAN/CAN_TX
- U501 pad 8: Net-(R501-Pad1) -> (no net)
- U501 pad 9: Net-(R503-Pad2) -> (no net)
Routing:
- net +3V3: track 503.4 -> 0.00 mm, vias 16 -> 0
- net +12V: track 206.9 -> 0.00 mm
- net /M_PRCHG: track 102.1 -> 0.00 mm, vias 6 -> 0
- net +5V: track 96.7 -> 0.00 mm, vias 4 -> 0
- net /FR_SW: track 94.7 -> 0.00 mm, vias 8 -> 0
- net /A_CNCTR: track 86.6 -> 0.00 mm, vias 4 -> 0
- net /A_PRCHG: track 82.6 -> 0.00 mm, vias 4 -> 0
- net /LEFT_SW: track 80.8 -> 0.00 mm, vias 4 -> 0
- net /M_CNCTR: track 77.6 -> 0.00 mm, vias 6 -> 0
- net /RIGHT_SW: track 74.7 -> 0.00 mm, vias 4 -> 0
- net /L_LGHT: track 66.9 -> 0.00 mm, vias 4 -> 0
- net Net-(J107-Pad16): track 65.7 -> 0.00 mm, vias 6 -> 0
- net Net-(J107-Pad17): track 65.0 -> 0.00 mm, vias 6 -> 0
- net /BPS_PWR: track 64.7 -> 0.00 mm
- net /CRUZ_ST: track 62.6 -> 0.00 mm, vias 2 -> 0
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- removed copper zone on B.Cu, net GND
- removed copper zone on F.Cu, net GND
- removed copper zone on B.Cu, net GNDPWR
- removed copper zone on F.Cu, net GNDPWR
Other:
- board outline removed
- board text removed: "12V"
- board text removed: "3V3"
- board text removed: "A-Contact"
- board text removed: "A-Precharge"
- board text removed: "Array Precharge LED"
- board text removed: "BPS Power"
- board text removed: "BPS Power LED"
- board text removed: "Backup"
- board text removed: "Backup Switch"
- board text removed: "BeVolt Dashboard V2 Designed by Chase Block Based on a design by Armin and Artin Taher UTSVT 2020"
- board text removed: "Brake Light"
- board text removed: "Brake-Pot"
- board text removed: "CLK"
- board text removed: "Cruise Enable"
- board text removed: "Cruise Set"
- board text removed: "Forward/Reverse"
- board text removed: "GND"
- board text removed: "Hazard Switch"
- board text removed: "Headlight"
- board text removed: "Headlight Switch"
- board text removed: "JTDI"
- board text removed: "JTDO"
- board text removed: "Kill Switch"
- board text removed: "Kill switch LED"
- board text removed: "Left Light"
- board text removed: "M-Contact"
- board text removed: "M-Precharge"
- board text removed: "Motor Contactor LED"
- board text removed: "Motor Precharge LED"
- board text removed: "Regen-Pot"
- board text removed: "Right Light"
- board text removed: "SWDIO"
- board text removed: "Turn Signal"
