File: Dashboard/Dash2/Dash2/PowerDist.sch (KiCad schematic (older format))
At the start: 15 parts, among them J301 CarPowerConnector, U301 RI3-1205S, U302 NCP1117-3.3_SOT223

Commit message: Add complete layout of the board
Parts:
- C301: Mouser Part Number (none) -> 80-C0805C475K3RAUTO
- C302, C304: Mouser Part Number (none) -> 80-C0805C106K8RAUTO
- C303: Mouser Part Number (none) -> 80-C0805C471J5HACTU
- D301: Mouser Part Number (none) -> 604-APTD2012LCGCK
- R301: Mouser Part Number (none) -> 71-CRCW08051K50FKEAC
- U301: Mouser Part Number (none) -> 919-RI3-1205S
- U302: Mouser Part Number (none) -> 863-NCP1117ST33T3G
Changed lines of the file:
@@
 EESchema Schematic File Version 4
-LIBS:Dash2-cache
-EELAYER 26 0
+EELAYER 30 0
 EELAYER END
 $Descr A4 11693 8268
@@
 F 2 "Capacitor_SMD:C_0805_2012Metric" H 2738 3250 50  0001 C CNN
 F 3 "~" H 2700 3400 50  0001 C CNN
+F 4 "80-C0805C475K3RAUTO " H 2700 3400 50  0001 C CNN "Mouser Part Number"
 	1    2700 3400
 	1    0    0    -1
@@
 F 3 "~" H 4550 2850 50  0001 C CNN
 F 4 "4kV" H 4550 2850 50  0001 C CNN "Rating"
+F 5 "80-C0805C471J5HACTU " H 4550 2850 50  0001 C CNN "Mouser Part Number"
 	1    4550 2850
 	0    -1   -1   0
@@
 F 4 "Green" V 6350 3600 50  0001 C CNN "Color"
 F 5 "APTD2012LCGCK" V 6350 3600 50  0001 C CNN "P/N"
+F 6 "604-APTD2012LCGCK " H 6350 3600 50  0001 C CNN "Mouser Part Number"
 	1    6350 3600
 	0    -1   -1   0
@@
 F 2 "Resistor_SMD:R_0805_2012Metric" V 6280 3250 50  0001 C CNN
 F 3 "~" H 6350 3250 50  0001 C CNN
+F 4 "71-CRCW08051K50FKEAC " H 6350 3250 50  0001 C CNN "Mouser Part Number"
 	1    6350 3250
 	1    0    0    -1
@@
 F 2 "Package_TO_SOT_SMD:SOT-223-3_TabPin2" H 4800 4700 50  0001 C CNN
 F 3 "http://www.onsemi.com/pub_link/Collateral/NCP1117-D.PDF" H 4900 4250 50  0001 C CNN
+F 4 "863-NCP1117ST33T3G " H 4800 4500 50  0001 C CNN "Mouser Part Number"
 	1    4800 4500
 	1    0    0    -1
@@
 F 2 "Capacitor_SMD:C_0805_2012Metric" H 4338 4550 50  0001 C CNN
 F 3 "~" H 4300 4700 50  0001 C CNN
+F 4 "80-C0805C106K8RAUTO " H 4300 4700 50  0001 C CNN "Mouser Part Number"
 	1    4300 4700
 	1    0    0    -1
@@
 F 2 "Capacitor_SMD:C_0805_2012Metric" H 5338 4550 50  0001 C CNN
 F 3 "~" H 5300 4700 50  0001 C CNN
+F 4 "80-C0805C106K8RAUTO " H 5300 4700 50  0001 C CNN "Mouser Part Number"
 	1    5300 4700
 	1    0    0    -1
@@
 F 2 "utsvt_ics:RI3_DC_Converter" H 4550 3200 50  0001 C CNN
 F 3 "" H 4550 3200 50  0001 C CNN
+F 4 "919-RI3-1205S " H 4550 3200 50  0001 C CNN "Mouser Part Number"
 	1    4550 3200
 	1    0    0    -1
