File: Dashboard/Dashboard/Dashboard.kicad_pcb (KiCad board)
At the start: 2 copper layers, 100 x 75 mm, 150 parts, among them J1 SWD, J10 Right Signal, J11 Brake Signal, J12 Headlight, J13 Vs-SPI3, J14 SPI3, J15 Vs-SPI1, J16 SPI1, J18 I2C3, J19 Switches-1, J2 Logic Analyzer, J20 Switches-2, J3 CarPowerConnector, J4 CAN_Out, J5 ContactorConnector, J6 ContactorConnector, J7 ContactorConnector, J8 ContactorConnector, J9 Left Signal, Q1 NVR4003NT3G, Q2 VND5N07-E, Q3 NVR4003NT3G, Q4 VND5N07-E, Q5 NVR4003NT3G, Q6 VND5N07-E, Q7 NVR4003NT3G, Q8 VND5N07-E, SW1 B3SL-1002P, U1 STM32F413RHTx, U10 SI8261ABC-IS, U11 BAS70-04, U12 SI8261ABC-IS, U13 BAS70-04, U14 SI8261ABC-IS, U15 BAS70-04, U2 RI3-1205S, U3 NCP1117-3.3_SOT223, U4 ADM3055E, U5 CDSOT23-T24CAN, U6 SI8261ABC-IS, U7 BAS70-04, U8 MAX6818EAP+, U9 MAX6818EAP+, Y1 NX8045GB-8.000M-STD-CSJ-1

Commit message: Make major changes to Dashboard and file structure.
Problem
=======
* The dashboard needs to be redesigned. These are continuing changes
to Dashboard 2.0.
* There are way too many files cluttering the Dashboard folder.
* We need to include LED indicators for the driver that make sense.

Solution
========
* I made major changes to the dashboard. These include the following:
  * Add an external LED board to mount on the steering wheel.
  * Add hardware timer circuitry for lights, so that the software does
    not have to concern itself with the flashers.
  * Generally cleaned up the dashboard's schematics
* There have also been changes made to the file system. All extra files
  that were not necessary have been removed. In the future, reference
  materials should be kept outside of version control.

Notes
=====
The dashboard still is not complete. We still need to address the following:
1. Pin assignments right now are mostly arbitrary. They are still subject to change.
2. The design needs to be verified.
3. We need to settle on the interface. Things like the ignition dial are still
   possible to change if we desire.
4. We need to add another potentiometer for the accelerator. This is missing because
   it was previously handled by the motor interface board.
5. Probably some other things that I'm forgetting.
Parts:
- removed C1, C3: 6pF, Capacitor_SMD:C_0805_2012Metric
- removed C10, C11, C12, C15, C19, C20, C24, C27, C31, C35, C39, C4, C5, C6, C7, C8: 0.1uF, Capacitor_SMD:C_0805_2012Metric
- removed C13, C14: 4.7uF, Capacitor_SMD:C_0805_2012Metric
- removed C16: 470pF, Capacitor_SMD:C_2220_5650Metric
- removed C17, C18, C22, C26, C30, C34, C38: 10uF, Capacitor_SMD:C_0805_2012Metric
- removed C2: 2.2uF, Capacitor_SMD:C_0805_2012Metric
- removed C21, C25: 0.01uF, Capacitor_SMD:C_0805_2012Metric
- removed C23: 0.22uF, Capacitor_SMD:C_0805_2012Metric
- removed C28, C29, C32, C33, C36, C37, C40, C41, C9: 1uF, Capacitor_SMD:C_0805_2012Metric
- removed C42: .1uF, Resistor_SMD:R_0805_2012Metric
- removed C43: 0.1uF, Resistor_SMD:R_0805_2012Metric
- removed D1: PowerOn, LED_SMD:LED_0805_2012Metric
- removed D2, D4, D6, D8: ContactorEn, LED_SMD:LED_0805_2012Metric
- removed D3, D5, D7, D9: 1N4148WS, Diode_SMD:D_SOD-323
- removed G***: LOGO, UTSVT_Special:UTSVT_Logo_Symbol
- removed J1: SWD, Connector_PinHeader_2.54mm:PinHeader_1x03_P2.54mm_Vertical
- removed J10: Right Signal, UTSVT_Connectors:Molex_MicroFit3.0_1x2xP3.00mm_PolarizingPeg_Vertical
- removed J11: Brake Signal, UTSVT_Connectors:Molex_MicroFit3.0_1x2xP3.00mm_PolarizingPeg_Vertical
- removed J12: Headlight, UTSVT_Connectors:Molex_MicroFit3.0_1x2xP3.00mm_PolarizingPeg_Vertical
- removed J13: Vs-SPI3, Connector_PinHeader_2.54mm:PinHeader_1x03_P2.54mm_Vertical
- removed J14: SPI3, Connector_Molex_Microfit:Molex_Micro-Fit_3.0_43650-0515_1x05_P3.00mm_Vertical
- removed J15: Vs-SPI1, Connector_PinHeader_2.54mm:PinHeader_1x03_P2.54mm_Vertical
- removed J16: SPI1, Connector_Molex_Microfit:Molex_Micro-Fit_3.0_43650-0515_1x05_P3.00mm_Vertical
- removed J18: I2C3, UTSVT_Connectors:Molex_MicroFit3.0_1x4xP3.00mm_PolarizingPeg_Vertical
- removed J19: Switches-1, Connector_Molex_Microfit:Molex_Micro-Fit_3.0_43045-1612_2x08_P3.00mm_Vertical
- removed J2: Logic Analyzer, Connector_PinHeader_2.54mm:PinHeader_2x05_P2.54mm_Vertical
- removed J20: Switches-2, Connector_Molex_Microfit:Molex_Micro-Fit_3.0_43045-1612_2x08_P3.00mm_Vertical
- removed J3: CarPowerConnector, UTSVT_Connectors:Molex_MicroFit3.0_1x2xP3.00mm_PolarizingPeg_Vertical
- removed J4: CAN_Out, UTSVT_Connectors:Molex_MicroFit3.0_1x4xP3.00mm_PolarizingPeg_Vertical
- removed J5, J6, J7, J8: ContactorConnector, UTSVT_Connectors:Molex_MicroFit3.0_1x4xP3.00mm_PolarizingPeg_Vertical
- removed J9: Left Signal, UTSVT_Connectors:Molex_MicroFit3.0_1x2xP3.00mm_PolarizingPeg_Vertical
- removed JP1: Termination Resistors, Connector_PinHeader_2.54mm:PinHeader_1x02_P2.54mm_Vertical
- removed L2, L3: 2kH, Inductor_SMD:L_0805_2012Metric
- removed L4: SRF0905-100Y, UTSVT_BPS:SRF0905A
- removed MH1, MH2, MH3, MH4: MountingHole, MountingHole:MountingHole_3mm
- removed Q1, Q3, Q5, Q7: NVR4003NT3G, Package_TO_SOT_SMD:SOT-23
- removed Q2, Q4, Q6, Q8: VND5N07-E, Package_TO_SOT_SMD:TO-252-2
- removed R1, R15, R23, R31, R7: 1.5k, Resistor_SMD:R_0805_2012Metric
- removed R10, R14, R18, R22, R26, R30, R34, R6: 100k, Resistor_SMD:R_0805_2012Metric
- removed R11, R19, R27, R35, R37, R38: 4.7k, Resistor_SMD:R_0805_2012Metric
- removed R12, R20, R28, R36: 1k, Resistor_SMD:R_0805_2012Metric
- removed R13, R17, R2, R21, R25, R29, R33, R5, R9: 0, Resistor_SMD:R_0805_2012Metric
- removed R16, R24, R32, R8: 470, Resistor_SMD:R_0805_2012Metric
- removed R3, R4: 60, Resistor_SMD:R_0805_2012Metric
- removed SW1: B3SL-1002P, Button_Switch_SMD:SW_SPST_B3SL-1002P
- removed TP1: +12V_TP, TestPoint:TestPoint_Keystone_5005-5009_Compact
- removed TP12, TP13, TP14, TP15: ContactorGate_TP, TestPoint:TestPoint_Keystone_5005-5009_Compact
- removed TP2: GNDPWR_TP, TestPoint:TestPoint_Keystone_5005-5009_Compact
- removed TP5: +3.3V_TP, TestPoint:TestPoint_Keystone_5005-5009_Compact
- removed U1: STM32F413RHTx, Package_QFP:LQFP-64_10x10mm_P0.5mm
- removed U10, U12, U14, U6: SI8261ABC-IS, Package_SO:SOIC-8_3.9x4.9mm_P1.27mm
- removed U11, U13, U15, U7: BAS70-04, Package_TO_SOT_SMD:SOT-23
- removed U2: RI3-1205S, UTSVT_ICs:RI3_DC_Converter
- removed U3: NCP1117-3.3_SOT223, Package_TO_SOT_SMD:SOT-223-3_TabPin2
- removed U4: ADM3055E, UTSVT_ICs:SOIC-20W_7.5x15.4mm_Pitch1.27mm
- removed U5: CDSOT23-T24CAN, Package_TO_SOT_SMD:SOT-23W
- removed U8, U9: MAX6818EAP+, footprints:MAX6818EAP&plus_
- removed Y1: NX8045GB-8.000M-STD-CSJ-1, UTSVT_BPS:NX8045GB-8.000M-STD-CSJ-1
Routing:
- net GND: track 422.2 -> 0.00 mm, vias 31 -> 0
- net +5V: track 324.1 -> 0.00 mm, vias 21 -> 0
- net +3V3: track 256.4 -> 0.00 mm, vias 11 -> 0
- net +12V: track 255.7 -> 0.00 mm, vias 15 -> 0
- net GNDPWR: track 186.2 -> 0.00 mm, vias 24 -> 0
- net /CAN1_RX: track 84.8 -> 0.00 mm, vias 2 -> 0
- net /CAN1_TX: track 81.6 -> 0.00 mm, vias 2 -> 0
- net /AC2_CHECK: track 79.1 -> 0.00 mm, vias 4 -> 0
- net /I2C3_SCL: track 77.0 -> 0.00 mm, vias 4 -> 0
- net /Headlight: track 75.2 -> 0.00 mm, vias 4 -> 0
- net /I2C3_SDA: track 72.2 -> 0.00 mm, vias 3 -> 0
- net /Left_Signal: track 70.9 -> 0.00 mm, vias 2 -> 0
- net /MC1_EN: track 69.9 -> 0.00 mm, vias 2 -> 0
- net /Right_Signal: track 61.8 -> 0.00 mm, vias 2 -> 0
- net /Brake_Signal: track 61.8 -> 0.00 mm, vias 3 -> 0
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- removed copper zone on F.Cu, net GND
- removed copper zone on B.Cu, net GNDPWR
Other:
- board outline removed
- net class Default: via_dia 0.8 -> 0.6; via_drill 0.4 -> 0.3
- board text removed: "Dashboard V1"
- board text removed: "Spring 2019: Nino Teruya"
