File: Dashboard/Dashboard/Dashboard.sch (KiCad schematic (older format))
At the start: 37 parts, among them J1 SWD, J10 Right Signal, J11 Brake Signal, J12 Headlight, J14 SPI3, J15 Vs-SPI1, J16 SPI1, J17 Vs-I2C3, J18 I2C3, J2 Logic Analyzer, J5 Array Contactor 1, J6 Motor Contactor 1, J7 Array Contactor 2, J8 Motor Contactor 2, J9 Left Signal, SW1 B3SL-1002P, U1 STM32F413RHTx, Y1 NX8045GB-8.000M-STD-CSJ-1

Commit message: Make major changes to Dashboard and file structure.
Problem
=======
* The dashboard needs to be redesigned. These are continuing changes
to Dashboard 2.0.
* There are way too many files cluttering the Dashboard folder.
* We need to include LED indicators for the driver that make sense.

Solution
========
* I made major changes to the dashboard. These include the following:
  * Add an external LED board to mount on the steering wheel.
  * Add hardware timer circuitry for lights, so that the software does
    not have to concern itself with the flashers.
  * Generally cleaned up the dashboard's schematics
* There have also been changes made to the file system. All extra files
  that were not necessary have been removed. In the future, reference
  materials should be kept outside of version control.

Notes
=====
The dashboard still is not complete. We still need to address the following:
1. Pin assignments right now are mostly arbitrary. They are still subject to change.
2. The design needs to be verified.
3. We need to settle on the interface. Things like the ignition dial are still
   possible to change if we desire.
4. We need to add another potentiometer for the accelerator. This is missing because
   it was previously handled by the motor interface board.
5. Probably some other things that I'm forgetting.
Parts:
- removed C1, C3: 6pF, Capacitor_SMD:C_0805_2012Metric, symbol Device:C
- removed C10, C11, C12, C4, C5, C6, C7, C8: 0.1uF, Capacitor_SMD:C_0805_2012Metric, symbol Device:C
- removed C13: 4.7uF, Capacitor_SMD:C_0805_2012Metric, symbol Device:C
- removed C2: 2.2uF, Capacitor_SMD:C_0805_2012Metric, symbol Device:C
- removed C9: 1uF, Capacitor_SMD:C_0805_2012Metric, symbol Device:C
- removed J1: SWD, Connector_PinHeader_2.54mm:PinHeader_1x03_P2.54mm_Vertical, symbol Connector_Generic:Conn_01x03
- removed J10: Right Signal, UTSVT_Connectors:Molex_MicroFit3.0_1x2xP3.00mm_PolarizingPeg_Vertical, symbol Connector_Generic:Conn_01x02
- removed J11: Brake Signal, UTSVT_Connectors:Molex_MicroFit3.0_1x2xP3.00mm_PolarizingPeg_Vertical, symbol Connector_Generic:Conn_01x02
- removed J12: Headlight, UTSVT_Connectors:Molex_MicroFit3.0_1x2xP3.00mm_PolarizingPeg_Vertical, symbol Connector_Generic:Conn_01x02
- removed J14: SPI3, Connector_Molex_Microfit:Molex_Micro-Fit_3.0_43650-0515_1x05_P3.00mm_Vertical, symbol Connector_Generic:Conn_01x05
- removed J15: Vs-SPI1, Connector_PinHeader_2.54mm:PinHeader_1x03_P2.54mm_Vertical, symbol Connector_Generic:Conn_01x03
- removed J16: SPI1, Connector_Molex_Microfit:Molex_Micro-Fit_3.0_43650-0515_1x05_P3.00mm_Vertical, symbol Connector_Generic:Conn_01x05
- removed J17: Vs-I2C3, Connector_PinHeader_2.54mm:PinHeader_1x03_P2.54mm_Vertical, symbol Connector_Generic:Conn_01x03
- removed J18: I2C3, UTSVT_Connectors:Molex_MicroFit3.0_1x4xP3.00mm_PolarizingPeg_Vertical, symbol Connector_Generic:Conn_01x04
- removed J2: Logic Analyzer, Connector_PinHeader_2.54mm:PinHeader_2x05_P2.54mm_Vertical, symbol Connector_Generic:Conn_02x05_Odd_Even
- removed J5: Array Contactor 1, UTSVT_Connectors:Molex_MicroFit3.0_1x4xP3.00mm_PolarizingPeg_Vertical, symbol Connector_Generic:Conn_01x04
- removed J6: Motor Contactor 1, UTSVT_Connectors:Molex_MicroFit3.0_1x4xP3.00mm_PolarizingPeg_Vertical, symbol Connector_Generic:Conn_01x04
- removed J7: Array Contactor 2, UTSVT_Connectors:Molex_MicroFit3.0_1x4xP3.00mm_PolarizingPeg_Vertical, symbol Connector_Generic:Conn_01x04
- removed J8: Motor Contactor 2, UTSVT_Connectors:Molex_MicroFit3.0_1x4xP3.00mm_PolarizingPeg_Vertical, symbol Connector_Generic:Conn_01x04
- removed J9: Left Signal, UTSVT_Connectors:Molex_MicroFit3.0_1x2xP3.00mm_PolarizingPeg_Vertical, symbol Connector_Generic:Conn_01x02
- removed MH1, MH2, MH3, MH4: MountingHole, MountingHole:MountingHole_3mm, symbol Mechanical:MountingHole
- removed R37, R38: 4.7k, Resistor_SMD:R_0805_2012Metric, symbol Device:R
- removed SW1: B3SL-1002P, Button_Switch_SMD:SW_SPST_B3SL-1002P, symbol Switch:SW_Push
- removed U1: STM32F413RHTx, Package_QFP:LQFP-64_10x10mm_P0.5mm, symbol MCU_ST_STM32F4:STM32F413RHTx
- removed Y1: NX8045GB-8.000M-STD-CSJ-1, UTSVT_BPS:NX8045GB-8.000M-STD-CSJ-1, symbol Device:Crystal
- added C101, C102, C103, C104: 1u, Capacitor_SMD:C_0805_2012Metric, symbol Device:C_Small
- added C105, C106, C109, C112, C113, C114, C115, C116, C117, C118, C119, C122, C123, C125: 100nF, Capacitor_SMD:C_0805_2012Metric, symbol Device:C
- added C107, C108: 4.3pF, Capacitor_SMD:C_0805_2012Metric, symbol Device:C
- added C110, C111: 2.2uF, Capacitor_SMD:C_0805_2012Metric, symbol Device:C_Small
- added C120, C121: 2pF, Capacitor_SMD:C_0805_2012Metric, symbol Device:C
- added C124: 4.7uF, Capacitor_SMD:C_0805_2012Metric, symbol Device:C
- added C126, C127: 0.1uF, Capacitor_SMD:C_0805_2012Metric, symbol Device:C
- added D102: LeftSignal, utsvt_conn:Molex_MicroFit3.0_1x2xP3.00mm_PolarizingPeg_Vertical, symbol Device:LED
- added D103: RightSignal, utsvt_conn:Molex_MicroFit3.0_1x2xP3.00mm_PolarizingPeg_Vertical, symbol Device:LED
- added D104: KILL_SW_LED, utsvt_conn:Molex_MicroFit3.0_1x2xP3.00mm_PolarizingPeg_Vertical, symbol Device:LED
- added D106: MOTOR-PRECHARGE, utsvt_conn:Molex_MicroFit3.0_1x2xP3.00mm_PolarizingPeg_Vertical, symbol Device:LED
- added D108: ARRAY-PRECHARGE, utsvt_conn:Molex_MicroFit3.0_1x2xP3.00mm_PolarizingPeg_Vertical, symbol Device:LED
- added D109, D110, D111, D112: D, Diode_SMD:D_0805_2012Metric, symbol Device:D
- added H101, H102, H103, H104, H105, H106, H107: MountingHole, MountingHole:MountingHole_3mm, symbol Mechanical:MountingHole
- added J1: LED_Cable, Connector_PinHeader_2.54mm:PinHeader_2x07_P2.54mm_Vertical, symbol Connector_Generic:Conn_01x11
- added J101: Left_Signal, utsvt_conn:Molex_MicroFit3.0_1x2xP3.00mm_PolarizingPeg_Vertical, symbol Connector_Generic:Conn_01x02
- added J102: Right_Signal, utsvt_conn:Molex_MicroFit3.0_1x2xP3.00mm_PolarizingPeg_Vertical, symbol Connector_Generic:Conn_01x02
- added J103: Brake Light, utsvt_conn:Molex_MicroFit3.0_1x2xP3.00mm_PolarizingPeg_Vertical, symbol Connector_Generic:Conn_01x02
- added J104: Headlight, utsvt_conn:Molex_MicroFit3.0_1x2xP3.00mm_PolarizingPeg_Vertical, symbol Connector_Generic:Conn_01x02
- added J105: Backup, utsvt_conn:Molex_MicroFit3.0_1x2xP3.00mm_PolarizingPeg_Vertical, symbol Connector_Generic:Conn_01x02
- added J106: BPS_PWR, utsvt_conn:Molex_MicroFit3.0_1x2xP3.00mm_PolarizingPeg_Vertical, symbol Connector_Generic:Conn_01x02
- added J107: Gecko_Cable, utsvt_conn:ribbon_cable_right_2x10, symbol Connector_Generic:Conn_02x10_Counter_Clockwise
- added J108: JTAG, Connector_PinHeader_2.54mm:PinHeader_1x06_P2.54mm_Vertical, symbol Connector_Generic:Conn_01x06
- added J109: Motor-C, utsvt_conn:Molex_MicroFit3.0_1x2xP3.00mm_PolarizingPeg_Vertical, symbol Connector_Generic:Conn_01x02
- added J110: Motor-P, utsvt_conn:Molex_MicroFit3.0_1x2xP3.00mm_PolarizingPeg_Vertical, symbol Connector_Generic:Conn_01x02
- added J111: Array-C, utsvt_conn:Molex_MicroFit3.0_1x2xP3.00mm_PolarizingPeg_Vertical, symbol Connector_Generic:Conn_01x02
- added J112: Array-P, utsvt_conn:Molex_MicroFit3.0_1x2xP3.00mm_PolarizingPeg_Vertical, symbol Connector_Generic:Conn_01x02
- added J113, J114: Conn_01x03_Female, utsvt_conn:Molex_MicroFit3.0_1x3xP3.00mm_PolarizingPeg_Vertical, symbol Connector_Generic:Conn_01x03
- added L101, L102, L103, L104: 22u, Inductor_SMD:L_0805_2012Metric, symbol pspice:INDUCTOR
- added PS101, PS102, PS103, PS104: RCD-24, utsvt_special:RCD-24, symbol Dash:RCD-24
- added Q1, Q2, Q3, Q4: Q_PNP_BCE, symbol Device:Q_PNP_BCE
- added R1, R2, R3: 100k, symbol Device:R_Small_US
- added R101, R102, R103, R107, R108, R116, R125, R126, R127, R128: 10k, Resistor_SMD:R_0805_2012Metric, symbol Device:R_US
- added R104, R105: 4.9k, Resistor_SMD:R_0805_2012Metric, symbol Device:R_US
- added R109, R110, R111, R112: 105, Resistor_SMD:R_0805_2012Metric, symbol Device:R_US
- added R113: 1.2k, Resistor_SMD:R_0805_2012Metric, symbol Device:R_US
- added R114, R115, R118, R120: 330R, Resistor_SMD:R_0805_2012Metric, symbol Device:R_US
- added R121, R122, R123, R124: 105R, Resistor_SMD:R_0805_2012Metric, symbol Device:R_US
- added SW101: CRUISE_SET, utsvt_conn:Molex_MicroFit3.0_1x3xP3.00mm_PolarizingPeg_Vertical, symbol Switch:SW_SPDT
- added SW102: CRUISE, utsvt_conn:Molex_MicroFit3.0_1x3xP3.00mm_PolarizingPeg_Vertical, symbol Switch:SW_SPDT
- added SW103: HAZARD, utsvt_conn:Molex_MicroFit3.0_1x3xP3.00mm_PolarizingPeg_Vertical, symbol Switch:SW_SPDT
- added SW104: HEADLIGHT_SW, utsvt_conn:Molex_MicroFit3.0_1x3xP3.00mm_PolarizingPeg_Vertical, symbol Switch:SW_SPDT
- added SW105: F/R_SW, utsvt_conn:Molex_MicroFit3.0_1x3xP3.00mm_PolarizingPeg_Vertical, symbol Switch:SW_SPDT
- added SW106: BACKUP_SW, utsvt_conn:Molex_MicroFit3.0_1x3xP3.00mm_PolarizingPeg_Vertical, symbol Switch:SW_SPDT
- added SW107: SW_Rotary2x6, utsvt_special:CK1035, symbol Switch:SW_Rotary2x6
- added SW108: TURN_SIGNAL_SW, utsvt_conn:Molex_MicroFit3.0_1x3xP3.00mm_PolarizingPeg_Vertical, symbol Switch:SW_SPDT_MSM
- added SW109: KILL_SW, utsvt_conn:Molex_MicroFit3.0_1x3xP3.00mm_PolarizingPeg_Vertical, symbol Switch:SW_SPDT
- added SW110: RESET, Button_Switch_SMD:SW_SPST_B3SL-1002P, symbol Switch:SW_SPST
- added TP101: POWER, TestPoint:TestPoint_Keystone_5005-5009_Compact, symbol Connector:TestPoint
- added U101, U102, U103, U104, U105, U106, U108, U109, U110, U111: EL3H7, Package_SO:SOP-4_4.4x2.6mm_P1.27mm, symbol Isolator:SFH617A-1
- added U107: STM32F413ZHTx, Package_QFP:LQFP-144_20x20mm_P0.5mm, symbol MCU_ST_STM32F4:STM32F413ZHTx
- added Y101: Crystal, Crystal:Crystal_SMD_TXC_7A-2Pin_5x3.2mm, symbol Device:Crystal
- added Y102: Crystal, Crystal:Crystal_SMD_TXC_9HT11-2Pin_2.0x1.2mm, symbol Device:Crystal
Connections:
- net labels added: +12V, A_CNCTR, A_PRCHG, BK_LGHT, BPS_FAULT, BPS_PWR, Backup, Brake_Pot, CRUZ_EN, CRUZ_ST, CTRL_FAULT, FR_SW, GNDA, GNDPWR, HZD_SW, HeadlightPWR, IG1, IG2, JTDI, JTDO, LEFT_BLINK, LEFT_SW, M_CNCTR, M_PRCHG, RIGHT_BLINK, RIGHT_SW, RSVD_LED, Regen_Pot
- net labels removed: AC1_CHECK, AC1_EN, AC2_CHECK, AC2_EN, Brake_Signal, CAN1_RX, CAN1_TX, Headlight, I2C3_SCL, I2C3_SDA, Left_Signal, MC1_CHECK, MC1_EN, MC2_CHECK, MC2_EN, OSC_IN, OSC_OUT, Right_Signal, SPI1_CLK, SPI1_MISO, SPI1_MOSI, SPI3_CLK, SPI3_MISO, SPI3_MOSI, UART1_RX, UART1_TX, array, bps, brake, chan1, chan2, cruise, decrease, hazard, increase, left, motor, regen, reverse, right, set-cancel, xtra1, xtra2, xtra3
- wire segments 230 -> 493
- no-connect marks 4 -> 101
Other:
- note added: "32K"
- note added: "8M"
- note added: "All of these are negative logic LEDs\n"
- note added: "Are there better/cheaper\ndrivers?"
- note added: "Exterior Lights"
- note added: "For the boad itself"
- note added: "For the gecko\n"
- note added: "Ignition Switch"
- note added: "Need to be LOW ESR\n"
- note added: "Potentiometers"
- note added: "Power state indicators"
- note added: "Should this be\nmale or female?"
- note added: "TODO: Assign pins for\n 1. BPS Fault\n 2. Control Fault\n 3. The Reserved Pin\nThe currently assigned pins should be considered temporary."
- note added: "TODO: Check to make sure\nthat all these switches have\nthe same "on" position."
- note added: "TODO: This connector was\noriginally the other way\naround. Will this still connect?"
- note added: "TODO: figure out which diodes\nthese are."
- note added: "TODO: make labels consistent.\nShould they be all UPPERCASE\nor Camel Case?"
- note added: "TODO: male or female?"
- note added: "TODO: should this be male or femal?"
- note added: "TODO: verify that this is all that needs to be done.\nRead the code to ensure all ports that are used are\non here.\n\nLook at all the other comments.\n\nAlso check over all the footprints again.\n\nAlso look at all the bodge wires running\naround the twins' board.\n\nAlso, if we're including another CAN line,\nwe should probably include another pot."
- note added: "These are negative-logic signals."
- note added: "Timing control for the lights"
- note added: "VDDA"
- note removed: "Bypass Capacitors"
- note removed: "Contactors"
- note removed: "Debug"
- note removed: "Header select\n"
- note removed: "I2C/SPI"
- note removed: "Isolated +5V and +3.3V.\nUse GND as common gnd for electronic components.\nConnect GNDPWR when using +12V."
- note removed: "Lights"
- note removed: "POWAH\n"
- note removed: "Place these capacitors as close to mcu as possible for correct operation.\nVDD/VSS"
- note removed: "Programming Pins."
- note removed: "SPI for screen. SPI for led. I2C incase"
- note removed: "Switches"
- note removed: "The crystal and caps have\nto be as close to the uC\nas possible."
- note removed: "VDDA/VSSA (VREF+/VREF-)"

Commit message: Change the MCU to the R (64-pin) variant.
Problem
=======
I don't want to have to solder 144 pins.

Solution
========
I changed the package of the MCU to the 64-pin
version, which now makes it the exact same as
the BPS.
Parts:
- removed C106, C114, C115, C116, C117, C118, C119, C122, C123: 100nF, Capacitor_SMD:C_0805_2012Metric, symbol Device:C
- removed C107, C108: 4.3pF, Capacitor_SMD:C_0805_2012Metric, symbol Device:C
- removed C110, C111: 2.2uF, Capacitor_SMD:C_0805_2012Metric, symbol Device:C_Small
- removed C120, C121: 2pF, Capacitor_SMD:C_0805_2012Metric, symbol Device:C
- removed J107: Gecko_Cable, utsvt_conn:ribbon_cable_right_2x10, symbol Connector_Generic:Conn_02x10_Counter_Clockwise
- removed J108: JTAG, Connector_PinHeader_2.54mm:PinHeader_1x06_P2.54mm_Vertical, symbol Connector_Generic:Conn_01x06
- removed PS101, PS102, PS103, PS104: RCD-24, utsvt_special:RCD-24, symbol Dash:RCD-24
- removed R116: 10k, Resistor_SMD:R_0805_2012Metric, symbol Device:R_US
- removed SW110: RESET, Button_Switch_SMD:SW_SPST_B3SL-1002P, symbol Switch:SW_SPST
- removed U107: STM32F413ZHTx, Package_QFP:LQFP-144_20x20mm_P0.5mm, symbol MCU_ST_STM32F4:STM32F413ZHTx
- removed Y101: Crystal, Crystal:Crystal_SMD_TXC_7A-2Pin_5x3.2mm, symbol Device:Crystal
- removed Y102: Crystal, Crystal:Crystal_SMD_TXC_9HT11-2Pin_2.0x1.2mm, symbol Device:Crystal
- added C3: 100nF, Capacitor_SMD:C_0805_2012Metric, symbol Device:C
- added C4, C5: 10pF, Capacitor_SMD:C_0805_2012Metric, symbol Device:C
- added C6: 4.7uF, symbol Device:C_Small
- added C7: 1uF, Capacitor_SMD:C_0805_2012Metric, symbol Device:C
- added J2: JTAG, Connector_PinHeader_2.54mm:PinHeader_1x06_P2.54mm_Vertical, symbol Connector_Generic:Conn_01x06
- added J3: Gecko_Cable, utsvt_conn:ribbon_cable_right_2x10, symbol Connector_Generic:Conn_02x10_Counter_Clockwise
- added PS1, PS2, PS3, PS4: RCD-24, symbol Dash:RCD-24
- added R6: 10k, Resistor_SMD:R_0805_2012Metric, symbol Device:R_US
- added SW1: RESET, Button_Switch_SMD:SW_SPST_B3SL-1002P, symbol Switch:SW_SPST
- added U1: STM32F413RHTx, Package_QFP:LQFP-64_10x10mm_P0.5mm, symbol MCU_ST_STM32F4:STM32F413RHTx
- added Y1: Crystal, Crystal:Crystal_SMD_TXC_7A-2Pin_5x3.2mm, symbol Device:Crystal
Connections:
- net +3V3: now also C7.1, J2.6 (Pin_6), J3.11 (Pin_11), U1.1 (VBAT), U1.13 (VDDA), U1.19 (VDD), U1.32 (VDD), U1.48 (VDD), U1.64 (VDD)
- net A_CNCTR: now also U1.23 (PA7), U1.59 (PB7)
- net A_PRCHG: now also U1.22 (PA6), U1.58 (PB6)
- net BK_LGHT: now also U1.14 (PA0)
- net BPS_FAULT: now also U1.52 (PC11)
- net Brake_Pot: now also U1.9 (PC1)
- net CRUZ_EN: now also U1.3 (PC14)
- net CRUZ_ST: now also U1.4 (PC15)
- net CTRL_FAULT: now also U1.53 (PC12)
- net FR_SW: now also U1.41 (PA8), U1.61 (PB8)
- net GND: now also C3.2, C4.2, C5.2, C6.1, C7.2, J2.5 (Pin_5), J3.1 (Pin_1), R6.2, SW1.1 (A), U1.12 (VSSA), U1.18 (VSS), U1.31 (VSS), U1.47 (VSS), U1.63 (VSS)
- net GNDPWR: now also PS1.4 (GND), PS2.4 (GND), PS3.4 (GND), PS4.4 (GND)
- net HeadlightPWR: now also U1.26 (PB0)
- net IG1: now also U1.35 (PB14), U1.42 (PA9)
- net IG2: now also U1.36 (PB15), U1.43 (PA10)
- net JTDI: now also J2.2 (Pin_2), U1.50 (PA15)
- net JTDO: now also J2.3 (Pin_3), U1.55 (PB3)
- net LEFT_SW: now also U1.28 (PB2)
- net M_CNCTR: now also U1.21 (PA5), U1.57 (PB5)
- net M_PRCHG: now also U1.20 (PA4), U1.56 (PB4)
- net NRST: now also C3.1, SW1.2 (B), U1.7 (NRST)
- net RIGHT_SW: now also U1.27 (PB1)
- net RSVD_LED: now also U1.2 (PC13)
- net SWCLK: now also J2.4 (Pin_4), U1.49 (PA14)
- net SWDIO: now also J2.1 (Pin_1), U1.46 (PA13)
- net at U103.3: now also PS1.3 (PWM)
- net at L101.1: now also PS1.1 (+Vin)
- net at J101.1 (Pin_1): now also PS1.5 (-Vout)
- net at J101.2 (Pin_2): now also PS1.6 (+Vout)
- net at U104.3: now also PS2.3 (PWM)
- net at L102.1: now also PS2.1 (+Vin)
- net at J102.1 (Pin_1): now also PS2.5 (-Vout)
- net at J102.2 (Pin_2): now also PS2.6 (+Vout)
- net at U105.3: now also PS3.3 (PWM)
- net at L103.1: now also PS3.1 (+Vin)
- net at J103.1 (Pin_1): now also PS3.5 (-Vout)
- net at J103.2 (Pin_2): now also PS3.6 (+Vout)
- net at U106.3: now also PS4.3 (PWM)
- net at L104.1: now also PS4.1 (+Vin)
- net at J104.1 (Pin_1): now also PS4.5 (-Vout)
- net at J104.2 (Pin_2): now also PS4.6 (+Vout)
- net Regen_Pot renamed Accel_Pot
- net Accel_Pot: now also U1.8 (PC0)
- new net: J3.17 (Pin_17), U1.16 (PA2)
- new net: J3.16 (Pin_16), U1.17 (PA3)
- new net: C6.2, U1.30 (VCAP_1)
- new net: C4.1, U1.5 (PH0), Y1.2
- new net: C5.1, U1.6 (PH1), Y1.1
- new net: R6.1, U1.60 (BOOT0)
- new net Car-CAN/CAN_RX: U1.44 (PA11)
- new net Car-CAN/CAN_TX: U1.45 (PA12)
- new net Motor-CAN/CAN_RX: U1.33 (PB12)
- new net Motor-CAN/CAN_TX: U1.34 (PB13)
- new net UART3_Tx: U1.29 (PB10)
- new net sheet5F7A9234/UART_RX: U1.25 (PC5)
- no-connect marks 101 -> 33
Other:
- note added: "TODO: verify that this is all that needs to be done.\nRead the code to ensure all ports that are used are\non here.\n\nLook at all the other comments.\n\nAlso check over all the footprints again.\n\nAlso look at all the bodge wires running\naround the twins' board."
- note removed: "32K"
- note removed: "Need to be LOW ESR\n"
- note removed: "TODO: verify that this is all that needs to be done.\nRead the code to ensure all ports that are used are\non here.\n\nLook at all the other comments.\n\nAlso check over all the footprints again.\n\nAlso look at all the bodge wires running\naround the twins' board.\n\nAlso, if we're including another CAN line,\nwe should probably include another pot."
- moved on the sheet: C105, C109, C112, C113, C124, C125

Commit message: Fixed minor issues and updated the pinout doc.
Connections:
- net A_CNCTR: no longer U1.23 (PA7)
- net A_PRCHG: no longer U1.22 (PA6)
- net FR_SW: no longer U1.41 (PA8)
- net IG1: no longer U1.42 (PA9)
- net IG2: no longer U1.43 (PA10)
- net M_CNCTR: no longer U1.21 (PA5)
- net M_PRCHG: no longer U1.20 (PA4)
- no-connect marks 33 -> 40
Changed lines of the file:
@@
 Brake_Pot
-Wire Wire Line
-	12450 6550 12850 6550
-Text Label 12850 6550 2    50   ~ 0
-FR_SW
-Wire Wire Line
-	12450 6150 12850 6150
-Wire Wire Line
-	12850 6250 12450 6250
-Wire Wire Line
-	12450 6350 12850 6350
-Wire Wire Line
-	12850 6450 12450 6450
-Text Label 12850 6150 2    50   ~ 0
-M_PRCHG
-Text Label 12850 6250 2    50   ~ 0
-M_CNCTR
-Text Label 12850 6350 2    50   ~ 0
-A_PRCHG
-Text Label 12850 6450 2    50   ~ 0
-A_CNCTR
-Wire Wire Line
-	12450 6650 12850 6650
-Wire Wire Line
-	12450 6750 12850 6750
-Text Label 12850 6650 2    50   ~ 0
-IG1
-Text Label 12850 6750 2    50   ~ 0
-IG2
 Wire Wire Line
 	12450 7550 12850 7550
@@
 $EndComp
 Connection ~ 2150 4350
+NoConn ~ 12450 6150
+NoConn ~ 12450 6250
+NoConn ~ 12450 6350
+NoConn ~ 12450 6450
+NoConn ~ 12450 6550
+NoConn ~ 12450 6650
+NoConn ~ 12450 6750
 $EndSCHEMATC

Commit message: Add redundant potentiometers and relabel components.
Parts:
- removed R125, R126: 10k, Resistor_SMD:R_0805_2012Metric, symbol Device:R_US
- added C16, C17: 0.1uF, Capacitor_SMD:C_0805_2012Metric, symbol Device:C
- added D4, D5, D6, D7: D, Diode_SMD:D_0805_2012Metric, symbol Device:D
- added J10, J11: Conn_01x03_Female, utsvt_conn:Molex_MicroFit3.0_1x3xP3.00mm_PolarizingPeg_Vertical, symbol Connector_Generic:Conn_01x03
- added R21, R22: 10k, Resistor_SMD:R_0805_2012Metric, symbol Device:R_US
- C10: renamed from C6; footprint (none) -> Capacitor_SMD:C_0805_2012Metric
- PS1, PS2, PS3, PS4: footprint (none) -> utsvt_special:RCD-24
- R15: renamed from R1; footprint (none) -> Resistor_SMD:R_0805_2012Metric
- R16: renamed from R2; footprint (none) -> Resistor_SMD:R_0805_2012Metric
- R17: renamed from R3; footprint (none) -> Resistor_SMD:R_0805_2012Metric
- renumbered C101 to C1, C112 to C11, C113 to C12, C124 to C13, C125 to C14, C7 to C15, C126 to C18, C127 to C19, C102 to C2, C103 to C3, C104 to C4, C3 to C5, C105 to C6, C4 to C7, C5 to C8, C109 to C9, D102 to D1, D109 to D10, D110 to D11, D111 to D12, D112 to D13, D103 to D2, D104 to D3, D106 to D8, D108 to D9, H101 to H1, H102 to H2, H103 to H3, H104 to H4, H105 to H5, H106 to H6, H107 to H7, J101 to J1, J109 to J12, J110 to J13, J111 to J14, J112 to J15, J113 to J16, J114 to J17, J102 to J2, J103 to J3, J104 to J4, J1 to J5, J105 to J6, J106 to J7, J2 to J8, J3 to J9, L101 to L1, L102 to L2, L103 to L3, L104 to L4, R101 to R1, R111 to R10, R112 to R11, R113 to R12, R114 to R13, R115 to R14, R6 to R18, R102 to R2, R118 to R23, R120 to R24, R121 to R25, R122 to R26, R123 to R27, R124 to R28, R103 to R3, R127 to R31, R128 to R32, R104 to R4, R105 to R5, R107 to R6, R108 to R7, R109 to R8, R110 to R9, SW101 to SW1, SW1 to SW10, SW102 to SW2, SW103 to SW3, SW104 to SW4, SW105 to SW5, SW106 to SW6, SW107 to SW7, SW108 to SW8, SW109 to SW9, TP101 to TP1, U101 to U1, U110 to U10, U111 to U11, U102 to U2, U103 to U3, U104 to U4, U105 to U5, U106 to U6, U1 to U7, U108 to U8, U109 to U9
Connections:
- net +3V3: now also D4.1 (K), D6.1 (K), J10.1 (Pin_1), J11.1 (Pin_1)
- net Accel_Pot: now also C16.1, D4.2 (A), D5.1 (K), R21.2; no longer C18.1, D10.2 (A), D11.1 (K), R31.2
- net Brake_Pot: now also C17.1, D6.2 (A), D7.1 (K), R22.2; no longer C19.1, D12.2 (A), D13.1 (K), R32.2
- net GND: now also C16.2, C17.2, D5.2 (A), D7.2 (A), J10.3 (Pin_3), J11.3 (Pin_3)
- net Accel_Pot2: now reaches U7.10 (PC2)
- net Accel_Pot2: now also C18.1, D10.2 (A), D11.1 (K), R31.2
- net Brake_Pot2: now reaches U7.11 (PC3)
- net Brake_Pot2: now also C19.1, D12.2 (A), D13.1 (K), R32.2
- new net: J10.2 (Pin_2), R21.1
- new net: J11.2 (Pin_2), R22.1
- no-connect marks 40 -> 38
