File: BPS/Master/CurrentBrdInterface.sch (KiCad schematic (older format))
At the start: 11 parts, among them J10 CurrentSlaveConnector, U5 LTC6256

Commit message: Reverts edited files that are not related to the FanBoard back to master branch's versions
Parts:
- U5: symbol BPSMaster-rescue:LTC6256-utsvt-bps -> utsvt-bps:LTC6256
Changed lines of the file:
@@
 The ADC has low impedence so buffer op-amp will prevent weird measurement deviations.
 $Comp
-L BPSMaster-rescue:LTC6256-utsvt-bps U5
+L utsvt-bps:LTC6256 U5
 U 1 1 5E3224B6
 P 3450 2850

Commit message: Created new sheet for bluetooth module. Using pins 37 and 38 of STM for UART communication with module. May need others to configure bluetooth module for low power mode.
Parts:
- U5: symbol utsvt-bps:LTC6256 -> BPSMaster-rescue:LTC6256-utsvt-bps
Changed lines of the file:
@@
 $Descr A4 11693 8268
 encoding utf-8
-Sheet 9 10
+Sheet 9 11
 Title ""
 Date ""
@@
 The ADC has low impedence so buffer op-amp will prevent weird measurement deviations.
 $Comp
-L utsvt-bps:LTC6256 U5
+L BPSMaster-rescue:LTC6256-utsvt-bps U5
 U 1 1 5E3224B6
 P 3450 2850
