File: BPS/Master/PowerDist.sch (KiCad schematic (older format))
At the start: 15 parts, among them J2 CarPowerConnector, U2 RI3-1205S, U3 NCP1117-3.3_SOT223

Commit message: Creates fan brd interface schematics and updates symbols/footprints related to the leader board
Parts:
- removed J2: CarPowerConnector, UTSVT_Connectors:Molex_MicroFit3.0_1x2xP3.00mm_PolarizingPeg_Vertical, symbol BPSMaster-rescue:CarPowerConnector-utsvt-connectors
- added J4: PowerConn, symbol Connector_Generic:Conn_01x02
- C12: renamed from C13; value 4.7uF -> 4.7u
- C13: renamed from C14; value 10uF -> 10u
- C14: renamed from C12; value 470pF -> 470p
- C15: value 10uF -> 10u
- L1: value 10uH -> 10u; symbol BPSMaster-rescue:SRF0905-100Y-utsvt-bps -> utsvt-bps:SRF0905-100Y
- U2: symbol BPSMaster-rescue:RI3-1205S-utsvt-power-regulators -> utsvt-power-regulators:RI3-1205S
- renumbered TP3 to TP2, TP5 to TP3, TP2 to TP4, TP4 to TP5
Connections:
- net +12V: now also J4.1 (Pin_1)
- net GNDPWR: now also J4.2 (Pin_2)
Other:
- note added: "+5V is already isolated so no need to isolate +3.3V"
- note removed: "Two separate converters would cause more noise on the board but less power waste.\nIf too much noise, add 5 to 3.3V regulator.\n"
- moved on the sheet: C13, C15, TP3, U3
