File: BPS/Master/PowerDist.sch (KiCad schematic (older format))
At the start: 15 parts, among them J4 PowerConn, U2 RI3-1205S, U3 NCP1117-3.3_SOT223

Commit message: Finishes schematics for bps leader board
Parts:
- J5: renamed from J4; footprint (none) -> Connector_Molex:Molex_Micro-Fit_3.0_43650-0215_1x02_P3.00mm_Vertical
Changed lines of the file:
@@
 $Descr A4 11693 8268
 encoding utf-8
-Sheet 2 10
+Sheet 2 11
 Title ""
 Date ""
@@
 $EndDescr
 $Comp
-L power:+12V #PWR018
+L power:+12V #PWR021
 U 1 1 5C35F2D2
 P 2450 3150
-F 0 "#PWR018" H 2450 3000 50  0001 C CNN
+F 0 "#PWR021" H 2450 3000 50  0001 C CNN
 F 1 "+12V" H 2465 3323 50  0000 C CNN
 F 2 "" H 2450 3150 50  0001 C CNN
@@
 +5V
 $Comp
-L power:+5V #PWR023
+L power:+5V #PWR026
 U 1 1 5C376123
 P 5200 3150
-F 0 "#PWR023" H 5200 3000 50  0001 C CNN
+F 0 "#PWR026" H 5200 3000 50  0001 C CNN
 F 1 "+5V" H 5215 3323 50  0000 C CNN
 F 2 "" H 5200 3150 50  0001 C CNN
@@
 	5500 3700 5500 3600
 $Comp
-L power:GND #PWR026
+L power:GND #PWR029
 U 1 1 5C58D746
 P 6350 3800
-F 0 "#PWR026" H 6350 3550 50  0001 C CNN
+F 0 "#PWR029" H 6350 3550 50  0001 C CNN
 F 1 "GND" H 6355 3627 50  0000 C CNN
 F 2 "" H 6350 3800 50  0001 C CNN
@@
 	6350 3450 6350 3400
 $Comp
-L power:+5V #PWR025
+L power:+5V #PWR028
 U 1 1 5C58FEF6
 P 6350 3050
-F 0 "#PWR025" H 6350 2900 50  0001 C CNN
+F 0 "#PWR028" H 6350 2900 50  0001 C CNN
 F 1 "+5V" H 6365 3223 50  0000 C CNN
 F 2 "" H 6350 3050 50  0001 C CNN
@@
 	6350 3050 6350 3100
 $Comp
-L power:GND #PWR024
+L power:GND #PWR027
 U 1 1 5C3F3B1F
 P 5200 3700
-F 0 "#PWR024" H 5200 3450 50  0001 C CNN
+F 0 "#PWR027" H 5200 3450 50  0001 C CNN
 F 1 "GND" H 5205 3527 50  0000 C CNN
 F 2 "" H 5200 3700 50  0001 C CNN
@@
 $EndComp
 $Comp
-L power:GNDPWR #PWR019
+L power:GNDPWR #PWR022
 U 1 1 5C3F7204
 P 2450 3650
-F 0 "#PWR019" H 2450 3450 50  0001 C CNN
+F 0 "#PWR022" H 2450 3450 50  0001 C CNN
 F 1 "GNDPWR" H 2454 3496 50  0000 C CNN
 F 2 "" H 2450 3600 50  0001 C CNN
@@
 $EndComp
 $Comp
-L power:+5V #PWR020
+L power:+5V #PWR023
 U 1 1 5C702374
 P 4050 4650
-F 0 "#PWR020" H 4050 4500 50  0001 C CNN
+F 0 "#PWR023" H 4050 4500 50  0001 C CNN
 F 1 "+5V" H 4065 4823 50  0000 C CNN
 F 2 "" H 4050 4650 50  0001 C CNN
@@
 	5050 4750 5050 4800
 $Comp
-L power:GND #PWR021
+L power:GND #PWR024
 U 1 1 5C703BF4
 P 4550 5200
-F 0 "#PWR021" H 4550 4950 50  0001 C CNN
+F 0 "#PWR024" H 4550 4950 50  0001 C CNN
 F 1 "GND" H 4555 5027 50  0000 C CNN
 F 2 "" H 4550 5200 50  0001 C CNN
@@
 Connection ~ 4050 4750
 $Comp
-L power:+3.3V #PWR022
+L power:+3.3V #PWR025
 U 1 1 5C7065C8
 P 5050 4650
-F 0 "#PWR022" H 5050 4500 50  0001 C CNN
+F 0 "#PWR025" H 5050 4500 50  0001 C CNN
 F 1 "+3.3V" H 5065 4823 50  0000 C CNN
 F 2 "" H 5050 4650 50  0001 C CNN
@@
 +5V is already isolated so no need to isolate +3.3V
 $Comp
-L Connector_Generic:Conn_01x02 J4
+L Connector_Generic:Conn_01x02 J5
 U 1 1 5F1149C6
 P 2150 3350
-F 0 "J4" H 2350 3400 50  0000 C CNN
+F 0 "J5" H 2350 3400 50  0000 C CNN
 F 1 "PowerConn" H 2450 3300 50  0000 C CNN
-F 2 "" H 2150 3350 50  0001 C CNN
+F 2 "Connector_Molex:Molex_Micro-Fit_3.0_43650-0215_1x02_P3.00mm_Vertical" H 2150 3350 50  0001 C CNN
 F 3 "~" H 2150 3350 50  0001 C CNN
 	1    2150 3350
