File: BPS/Master/FanBrdInterface.sch (KiCad schematic (older format))
At the start: 15 parts, among them J11 FanBrdConn, U14 SI8261ABC-IS, U15 SI8261ABC-IS, U16 SI8261ABC-IS, U17 SI8261ABC-IS

Commit message: Finishes schematics for bps leader board
Parts:
- renumbered J11 to J12
Changed lines of the file:
@@
 $Descr A4 11693 8268
 encoding utf-8
-Sheet 10 10
+Sheet 10 11
 Title ""
 Date ""
@@
 P 4100 1750
 AR Path="/5C38C674/5F130099" Ref="#PWR?"  Part="1"
-AR Path="/5F145F02/5F130099" Ref="#PWR082"  Part="1"
-F 0 "#PWR?" H 4100 1600 50  0001 C CNN
+AR Path="/5F145F02/5F130099" Ref="#PWR085"  Part="1"
+F 0 "#PWR085" H 4100 1600 50  0001 C CNN
 F 1 "+12V" H 4115 1923 50  0000 C CNN
 F 2 "" H 4100 1750 50  0001 C CNN
@@
 AR Path="/5C38C674/5F13009F" Ref="C?"  Part="1"
 AR Path="/5F145F02/5F13009F" Ref="C38"  Part="1"
-F 0 "C?" H 4215 2046 50  0000 L CNN
+F 0 "C38" H 4215 2046 50  0000 L CNN
 F 1 "10u" H 4215 1955 50  0000 L CNN
 F 2 "Capacitor_SMD:C_0805_2012Metric" H 4138 1850 50  0001 C CNN
@@
 AR Path="/5C38C674/5F1300A5" Ref="C?"  Part="1"
 AR Path="/5F145F02/5F1300A5" Ref="C39"  Part="1"
-F 0 "C?" H 4665 2046 50  0000 L CNN
+F 0 "C39" H 4665 2046 50  0000 L CNN
 F 1 "0.1u" H 4665 1955 50  0000 L CNN
 F 2 "Capacitor_SMD:C_0805_2012Metric" H 4588 1850 50  0001 C CNN
@@
 P 4100 2250
 AR Path="/5C38C674/5F1300F5" Ref="#PWR?"  Part="1"
-AR Path="/5F145F02/5F1300F5" Ref="#PWR083"  Part="1"
-F 0 "#PWR?" H 4100 2050 50  0001 C CNN
+AR Path="/5F145F02/5F1300F5" Ref="#PWR086"  Part="1"
+F 0 "#PWR086" H 4100 2050 50  0001 C CNN
 F 1 "GNDPWR" H 4104 2096 50  0000 C CNN
 F 2 "" H 4100 2200 50  0001 C CNN
@@
 P 4900 3000
 AR Path="/5C38C674/5F1300FB" Ref="#PWR?"  Part="1"
-AR Path="/5F145F02/5F1300FB" Ref="#PWR084"  Part="1"
-F 0 "#PWR?" H 4900 2800 50  0001 C CNN
+AR Path="/5F145F02/5F1300FB" Ref="#PWR087"  Part="1"
+F 0 "#PWR087" H 4900 2800 50  0001 C CNN
 F 1 "GNDPWR" H 4904 2846 50  0000 C CNN
 F 2 "" H 4900 2950 50  0001 C CNN
@@
 	4900 2700 4900 2800
 $Comp
-L power:GND #PWR078
+L power:GND #PWR081
 U 1 1 5F1328D9
 P 3700 3000
-F 0 "#PWR?" H 3700 2750 50  0001 C CNN
+F 0 "#PWR081" H 3700 2750 50  0001 C CNN
 F 1 "GND" H 3705 2827 50  0000 C CNN
 F 2 "" H 3700 3000 50  0001 C CNN
@@
 U 1 1 5F14B1DD
 P 4300 2500
-F 0 "U?" H 4300 1850 50  0000 C CNN
+F 0 "U14" H 4300 1850 50  0000 C CNN
 F 1 "SI8261ABC-IS" H 4300 1950 50  0000 C CNN
 F 2 "Package_SO:SOIC-8_3.9x4.9mm_P1.27mm" H 4300 2500 50  0001 C CNN
@@
 U 1 1 5F14C350
 P 3450 2700
-F 0 "R?" V 3350 2700 50  0000 C CNN
+F 0 "R38" V 3350 2700 50  0000 C CNN
 F 1 "117" V 3450 2700 50  0000 C CNN
 F 2 "Resistor_SMD:R_0805_2012Metric" V 3380 2700 50  0001 C CNN
@@
 	3100 2700 3300 2700
 $Comp
-L Connector_Generic:Conn_02x03_Top_Bottom J11
+L Connector_Generic:Conn_02x03_Top_Bottom J12
 U 1 1 5F14E9E0
 P 7600 4050
-F 0 "J?" H 7650 4367 50  0000 C CNN
+F 0 "J12" H 7650 4367 50  0000 C CNN
 F 1 "FanBrdConn" H 7650 4276 50  0000 C CNN
 F 2 "Connector_Molex:Molex_Micro-Fit_3.0_43045-0612_2x03_P3.00mm_Vertical" H 7600 4050 50  0001 C CNN
@@
 P 4900 3750
 AR Path="/5C38C674/5F1531CC" Ref="#PWR?"  Part="1"
-AR Path="/5F145F02/5F1531CC" Ref="#PWR085"  Part="1"
-F 0 "#PWR?" H 4900 3600 50  0001 C CNN
+AR Path="/5F145F02/5F1531CC" Ref="#PWR088"  Part="1"
+F 0 "#PWR088" H 4900 3600 50  0001 C CNN
 F 1 "+12V" H 4915 3923 50  0000 C CNN
 F 2 "" H 4900 3750 50  0001 C CNN
@@
 P 4900 4250
 AR Path="/5C38C674/5F1531F5" Ref="#PWR?"  Part="1"
-AR Path="/5F145F02/5F1531F5" Ref="#PWR086"  Part="1"
-F 0 "#PWR?" H 4900 4050 50  0001 C CNN
+AR Path="/5F145F02/5F1531F5" Ref="#PWR089"  Part="1"
+F 0 "#PWR089" H 4900 4050 50  0001 C CNN
 F 1 "GNDPWR" H 4904 4096 50  0000 C CNN
 F 2 "" H 4900 4200 50  0001 C CNN
@@
 	4900 3950 4900 4050
 $Comp
-L power:GND #PWR079
+L power:GND #PWR082
 U 1 1 5F1531FD
 P 3700 4250
-F 0 "#PWR?" H 3700 4000 50  0001 C CNN
+F 0 "#PWR082" H 3700 4000 50  0001 C CNN
 F 1 "GND" H 3705 4077 50  0000 C CNN
 F 2 "" H 3700 4250 50  0001 C CNN
@@
 U 1 1 5F153207
 P 4300 3750
-F 0 "U?" H 4300 3100 50  0000 C CNN
+F 0 "U15" H 4300 3100 50  0000 C CNN
 F 1 "SI8261ABC-IS" H 4300 3200 50  0000 C CNN
 F 2 "Package_SO:SOIC-8_3.9x4.9mm_P1.27mm" H 4300 3750 50  0001 C CNN
@@
 U 1 1 5F15320D
 P 3450 3950
-F 0 "R?" V 3350 3950 50  0000 C CNN
+F 0 "R39" V 3350 3950 50  0000 C CNN
 F 1 "117" V 3450 3950 50  0000 C CNN
 F 2 "Resistor_SMD:R_0805_2012Metric" V 3380 3950 50  0001 C CNN
@@
 P 4900 5000
 AR Path="/5C38C674/5F155440" Ref="#PWR?"  Part="1"
-AR Path="/5F145F02/5F155440" Ref="#PWR087"  Part="1"
-F 0 "#PWR?" H 4900 4850 50  0001 C CNN
+AR Path="/5F145F02/5F155440" Ref="#PWR090"  Part="1"
+F 0 "#PWR090" H 4900 4850 50  0001 C CNN
 F 1 "+12V" H 4915 5173 50  0000 C CNN
 F 2 "" H 4900 5000 50  0001 C CNN
@@
 P 4900 5500
 AR Path="/5C38C674/5F155469" Ref="#PWR?"  Part="1"
-AR Path="/5F145F02/5F155469" Ref="#PWR088"  Part="1"
-F 0 "#PWR?" H 4900 5300 50  0001 C CNN
+AR Path="/5F145F02/5F155469" Ref="#PWR091"  Part="1"
+F 0 "#PWR091" H 4900 5300 50  0001 C CNN
 F 1 "GNDPWR" H 4904 5346 50  0000 C CNN
 F 2 "" H 4900 5450 50  0001 C CNN
@@
 	4900 5200 4900 5300
 $Comp
-L power:GND #PWR080
+L power:GND #PWR083
 U 1 1 5F155471
 P 3700 5500
-F 0 "#PWR?" H 3700 5250 50  0001 C CNN
+F 0 "#PWR083" H 3700 5250 50  0001 C CNN
 F 1 "GND" H 3705 5327 50  0000 C CNN
 F 2 "" H 3700 5500 50  0001 C CNN
@@
 U 1 1 5F15547B
 P 4300 5000
-F 0 "U?" H 4300 4350 50  0000 C CNN
+F 0 "U16" H 4300 4350 50  0000 C CNN
 F 1 "SI8261ABC-IS" H 4300 4450 50  0000 C CNN
 F 2 "Package_SO:SOIC-8_3.9x4.9mm_P1.27mm" H 4300 5000 50  0001 C CNN
@@
 U 1 1 5F155481
 P 3450 5200
-F 0 "R?" V 3350 5200 50  0000 C CNN
+F 0 "R40" V 3350 5200 50  0000 C CNN
 F 1 "117" V 3450 5200 50  0000 C CNN
 F 2 "Resistor_SMD:R_0805_2012Metric" V 3380 5200 50  0001 C CNN
@@
 FAN3
 $Comp
-L power:+12V #PWR094
+L power:+12V #PWR097
 U 1 1 5F157D4C
 P 7300 3850
-F 0 "#PWR?" H 7300 3700 50  0001 C CNN
+F 0 "#PWR097" H 7300 3700 50  0001 C CNN
 F 1 "+12V" H 7315 4023 50  0000 C CNN
 F 2 "" H 7300 3850 50  0001 C CNN
@@
 P 8000 4250
 AR Path="/5C38C674/5F15A290" Ref="#PWR?"  Part="1"
-AR Path="/5F145F02/5F15A290" Ref="#PWR096"  Part="1"
-F 0 "#PWR?" H 8000 4050 50  0001 C CNN
+AR Path="/5F145F02/5F15A290" Ref="#PWR099"  Part="1"
+F 0 "#PWR099" H 8000 4050 50  0001 C CNN
 F 1 "GNDPWR" H 8004 4096 50  0000 C CNN
 F 2 "" H 8000 4200 50  0001 C CNN
@@
 P 4900 6250
 AR Path="/5C38C674/5F1644DE" Ref="#PWR?"  Part="1"
-AR Path="/5F145F02/5F1644DE" Ref="#PWR089"  Part="1"
-F 0 "#PWR?" H 4900 6100 50  0001 C CNN
+AR Path="/5F145F02/5F1644DE" Ref="#PWR092"  Part="1"
+F 0 "#PWR092" H 4900 6100 50  0001 C CNN
 F 1 "+12V" H 4915 6423 50  0000 C CNN
 F 2 "" H 4900 6250 50  0001 C CNN
@@
 P 4900 6750
 AR Path="/5C38C674/5F164507" Ref="#PWR?"  Part="1"
-AR Path="/5F145F02/5F164507" Ref="#PWR090"  Part="1"
-F 0 "#PWR?" H 4900 6550 50  0001 C CNN
+AR Path="/5F145F02/5F164507" Ref="#PWR093"  Part="1"
+F 0 "#PWR093" H 4900 6550 50  0001 C CNN
 F 1 "GNDPWR" H 4904 6596 50  0000 C CNN
 F 2 "" H 4900 6700 50  0001 C CNN
@@
 	4900 6450 4900 6550
 $Comp
-L power:GND #PWR081
+L power:GND #PWR084
 U 1 1 5F16450F
 P 3700 6750
-F 0 "#PWR?" H 3700 6500 50  0001 C CNN
+F 0 "#PWR084" H 3700 6500 50  0001 C CNN
 F 1 "GND" H 3705 6577 50  0000 C CNN
 F 2 "" H 3700 6750 50  0001 C CNN
@@
 U 1 1 5F164519
 P 4300 6250
-F 0 "U?" H 4300 5600 50  0000 C CNN
+F 0 "U17" H 4300 5600 50  0000 C CNN
 F 1 "SI8261ABC-IS" H 4300 5700 50  0000 C CNN
 F 2 "Package_SO:SOIC-8_3.9x4.9mm_P1.27mm" H 4300 6250 50  0001 C CNN
@@
 U 1 1 5F16451F
 P 3450 6450
-F 0 "R?" V 3350 6450 50  0000 C CNN
+F 0 "R41" V 3350 6450 50  0000 C CNN
 F 1 "117" V 3450 6450 50  0000 C CNN
 F 2 "Resistor_SMD:R_0805_2012Metric" V 3380 6450 50  0001 C CNN
@@
 U 1 1 5F1A07F9
 P 7300 4400
-F 0 "C?" H 7415 4446 50  0000 L CNN
+F 0 "C43" H 7415 4446 50  0000 L CNN
 F 1 "0.1u" H 7415 4355 50  0000 L CNN
 F 2 "Capacitor_SMD:C_0805_2012Metric" H 7338 4250 50  0001 C CNN
@@
 P 7300 4650
 AR Path="/5C38C674/5F1A1FAF" Ref="#PWR?"  Part="1"
-AR Path="/5F145F02/5F1A1FAF" Ref="#PWR095"  Part="1"
-F 0 "#PWR?" H 7300 4450 50  0001 C CNN
+AR Path="/5F145F02/5F1A1FAF" Ref="#PWR098"  Part="1"
+F 0 "#PWR098" H 7300 4450 50  0001 C CNN
 F 1 "GNDPWR" H 7304 4496 50  0000 C CNN
 F 2 "" H 7300 4600 50  0001 C CNN
@@
 AR Path="/5C38C674/5F1CC902" Ref="C?"  Part="1"
 AR Path="/5F145F02/5F1CC902" Ref="C40"  Part="1"
-F 0 "C?" H 5265 3896 50  0000 L CNN
+F 0 "C40" H 5265 3896 50  0000 L CNN
 F 1 "0.1u" H 5265 3805 50  0000 L CNN
 F 2 "Capacitor_SMD:C_0805_2012Metric" H 5188 3700 50  0001 C CNN
@@
 AR Path="/5C38C674/5F1CE8B4" Ref="C?"  Part="1"
 AR Path="/5F145F02/5F1CE8B4" Ref="C41"  Part="1"
-F 0 "C?" H 5265 5146 50  0000 L CNN
+F 0 "C41" H 5265 5146 50  0000 L CNN
 F 1 "0.1u" H 5265 5055 50  0000 L CNN
 F 2 "Capacitor_SMD:C_0805_2012Metric" H 5188 4950 50  0001 C CNN
@@
 AR Path="/5C38C674/5F1D0348" Ref="C?"  Part="1"
 AR Path="/5F145F02/5F1D0348" Ref="C42"  Part="1"
-F 0 "C?" H 5265 6396 50  0000 L CNN
+F 0 "C42" H 5265 6396 50  0000 L CNN
 F 1 "0.1u" H 5265 6305 50  0000 L CNN
 F 2 "Capacitor_SMD:C_0805_2012Metric" H 5188 6200 50  0001 C CNN
@@
 P 5400 6350
 AR Path="/5C38C674/5F1D20B3" Ref="#PWR?"  Part="1"
-AR Path="/5F145F02/5F1D20B3" Ref="#PWR093"  Part="1"
-F 0 "#PWR?" H 5400 6150 50  0001 C CNN
+AR Path="/5F145F02/5F1D20B3" Ref="#PWR096"  Part="1"
+F 0 "#PWR096" H 5400 6150 50  0001 C CNN
 F 1 "GNDPWR" H 5404 6196 50  0000 C CNN
 F 2 "" H 5400 6300 50  0001 C CNN
@@
 P 5400 5100
 AR Path="/5C38C674/5F1D596F" Ref="#PWR?"  Part="1"
-AR Path="/5F145F02/5F1D596F" Ref="#PWR092"  Part="1"
-F 0 "#PWR?" H 5400 4900 50  0001 C CNN
+AR Path="/5F145F02/5F1D596F" Ref="#PWR095"  Part="1"
+F 0 "#PWR095" H 5400 4900 50  0001 C CNN
 F 1 "GNDPWR" H 5404 4946 50  0000 C CNN
 F 2 "" H 5400 5050 50  0001 C CNN
@@
 P 5300 3850
 AR Path="/5C38C674/5F1DA30D" Ref="#PWR?"  Part="1"
-AR Path="/5F145F02/5F1DA30D" Ref="#PWR091"  Part="1"
-F 0 "#PWR?" H 5300 3650 50  0001 C CNN
+AR Path="/5F145F02/5F1DA30D" Ref="#PWR094"  Part="1"
+F 0 "#PWR094" H 5300 3650 50  0001 C CNN
 F 1 "GNDPWR" H 5304 3696 50  0000 C CNN
 F 2 "" H 5300 3800 50  0001 C CNN
