File: BPS/Master/SensorBrdInterface.sch (KiCad schematic (older format))
At the start: 15 parts, among them J5 MinionConn, J6 CurrentConn, U5 LTC6820, U6 LTC6820, U7 HX1188FNL

Commit message: Finishes schematics for bps leader board
Parts:
- J7: renamed from J6; footprint (none) -> Connector_Molex:Molex_Micro-Fit_3.0_43650-0415_1x04_P3.00mm_Vertical
- renumbered J5 to J6
Changed lines of the file:
@@
 $Descr A4 11693 8268
 encoding utf-8
-Sheet 5 10
+Sheet 5 11
 Title ""
 Date ""
@@
 P 4650 2800
 AR Path="/5C4C7509/5D76E53B" Ref="#PWR?"  Part="1"
-AR Path="/5D766247/5D76E53B" Ref="#PWR038"  Part="1"
-F 0 "#PWR038" H 4650 2550 50  0001 C CNN
+AR Path="/5D766247/5D76E53B" Ref="#PWR041"  Part="1"
+F 0 "#PWR041" H 4650 2550 50  0001 C CNN
 F 1 "GND" H 4655 2627 50  0000 C CNN
 F 2 "" H 4650 2800 50  0001 C CNN
@@
 P 2550 2550
 AR Path="/5C4C7509/5D76E546" Ref="#PWR?"  Part="1"
-AR Path="/5D766247/5D76E546" Ref="#PWR036"  Part="1"
-F 0 "#PWR036" H 2550 2300 50  0001 C CNN
+AR Path="/5D766247/5D76E546" Ref="#PWR039"  Part="1"
+F 0 "#PWR039" H 2550 2300 50  0001 C CNN
 F 1 "GND" V 2555 2422 50  0000 R CNN
 F 2 "" H 2550 2550 50  0001 C CNN
@@
 P 2050 3450
 AR Path="/5C4C7509/5D76E556" Ref="#PWR?"  Part="1"
-AR Path="/5D766247/5D76E556" Ref="#PWR033"  Part="1"
-F 0 "#PWR033" H 2050 3200 50  0001 C CNN
+AR Path="/5D766247/5D76E556" Ref="#PWR036"  Part="1"
+F 0 "#PWR036" H 2050 3200 50  0001 C CNN
 F 1 "GND" H 2055 3277 50  0000 C CNN
 F 2 "" H 2050 3450 50  0001 C CNN
@@
 P 4850 3650
 AR Path="/5C4C7509/5D76E575" Ref="#PWR?"  Part="1"
-AR Path="/5D766247/5D76E575" Ref="#PWR041"  Part="1"
-F 0 "#PWR041" H 4850 3400 50  0001 C CNN
+AR Path="/5D766247/5D76E575" Ref="#PWR044"  Part="1"
+F 0 "#PWR044" H 4850 3400 50  0001 C CNN
 F 1 "GND" H 4855 3477 50  0000 C CNN
 F 2 "" H 4850 3650 50  0001 C CNN
@@
 P 5100 2650
 AR Path="/5C4C7509/5D76E58F" Ref="#PWR?"  Part="1"
-AR Path="/5D766247/5D76E58F" Ref="#PWR044"  Part="1"
-F 0 "#PWR044" H 5100 2400 50  0001 C CNN
+AR Path="/5D766247/5D76E58F" Ref="#PWR047"  Part="1"
+F 0 "#PWR047" H 5100 2400 50  0001 C CNN
 F 1 "GND" V 5105 2522 50  0000 R CNN
 F 2 "" H 5100 2650 50  0001 C CNN
@@
 P 9400 3500
 AR Path="/5C4C7509/5D76E59D" Ref="J?"  Part="1"
-AR Path="/5D766247/5D76E59D" Ref="J5"  Part="1"
-F 0 "J5" H 9479 3492 50  0000 L CNN
+AR Path="/5D766247/5D76E59D" Ref="J6"  Part="1"
+F 0 "J6" H 9479 3492 50  0000 L CNN
 F 1 "MinionConn" H 9479 3401 50  0000 L CNN
 F 2 "UTSVT_Connectors:Molex_MicroFit3.0_1x2xP3.00mm_PolarizingPeg_Vertical" H 9400 3500 50  0001 C CNN
@@
 P 4850 3200
 AR Path="/5C4C7509/5D76E5AC" Ref="#PWR?"  Part="1"
-AR Path="/5D766247/5D76E5AC" Ref="#PWR040"  Part="1"
-F 0 "#PWR040" H 4850 3050 50  0001 C CNN
+AR Path="/5D766247/5D76E5AC" Ref="#PWR043"  Part="1"
+F 0 "#PWR043" H 4850 3050 50  0001 C CNN
 F 1 "+5V" H 4865 3373 50  0000 C CNN
 F 2 "" H 4850 3200 50  0001 C CNN
@@
 P 2050 3000
 AR Path="/5C4C7509/5D76E5D1" Ref="#PWR?"  Part="1"
-AR Path="/5D766247/5D76E5D1" Ref="#PWR032"  Part="1"
-F 0 "#PWR032" H 2050 2850 50  0001 C CNN
+AR Path="/5D766247/5D76E5D1" Ref="#PWR035"  Part="1"
+F 0 "#PWR035" H 2050 2850 50  0001 C CNN
 F 1 "+5V" H 2065 3173 50  0000 C CNN
 F 2 "" H 2050 3000 50  0001 C CNN
@@
 P 4650 5050
 AR Path="/5C4C7509/5F151E6E" Ref="#PWR?"  Part="1"
-AR Path="/5D766247/5F151E6E" Ref="#PWR039"  Part="1"
-F 0 "#PWR039" H 4650 4800 50  0001 C CNN
+AR Path="/5D766247/5F151E6E" Ref="#PWR042"  Part="1"
+F 0 "#PWR042" H 4650 4800 50  0001 C CNN
 F 1 "GND" H 4655 4877 50  0000 C CNN
 F 2 "" H 4650 5050 50  0001 C CNN
@@
 P 2550 4800
 AR Path="/5C4C7509/5F151E76" Ref="#PWR?"  Part="1"
-AR Path="/5D766247/5F151E76" Ref="#PWR037"  Part="1"
-F 0 "#PWR037" H 2550 4550 50  0001 C CNN
+AR Path="/5D766247/5F151E76" Ref="#PWR040"  Part="1"
+F 0 "#PWR040" H 2550 4550 50  0001 C CNN
 F 1 "GND" V 2555 4672 50  0000 R CNN
 F 2 "" H 2550 4800 50  0001 C CNN
@@
 P 2050 5700
 AR Path="/5C4C7509/5F151E86" Ref="#PWR?"  Part="1"
-AR Path="/5D766247/5F151E86" Ref="#PWR035"  Part="1"
-F 0 "#PWR035" H 2050 5450 50  0001 C CNN
+AR Path="/5D766247/5F151E86" Ref="#PWR038"  Part="1"
+F 0 "#PWR038" H 2050 5450 50  0001 C CNN
 F 1 "GND" H 2055 5527 50  0000 C CNN
 F 2 "" H 2050 5700 50  0001 C CNN
@@
 P 4850 5900
 AR Path="/5C4C7509/5F151EA5" Ref="#PWR?"  Part="1"
-AR Path="/5D766247/5F151EA5" Ref="#PWR043"  Part="1"
-F 0 "#PWR043" H 4850 5650 50  0001 C CNN
+AR Path="/5D766247/5F151EA5" Ref="#PWR046"  Part="1"
+F 0 "#PWR046" H 4850 5650 50  0001 C CNN
 F 1 "GND" H 4855 5727 50  0000 C CNN
 F 2 "" H 4850 5900 50  0001 C CNN
@@
 P 5100 4900
 AR Path="/5C4C7509/5F151EBF" Ref="#PWR?"  Part="1"
-AR Path="/5D766247/5F151EBF" Ref="#PWR045"  Part="1"
-F 0 "#PWR045" H 5100 4650 50  0001 C CNN
+AR Path="/5D766247/5F151EBF" Ref="#PWR048"  Part="1"
+F 0 "#PWR048" H 5100 4650 50  0001 C CNN
 F 1 "GND" V 5105 4772 50  0000 R CNN
 F 2 "" H 5100 4900 50  0001 C CNN
@@
 P 4850 5450
 AR Path="/5C4C7509/5F151EC9" Ref="#PWR?"  Part="1"
-AR Path="/5D766247/5F151EC9" Ref="#PWR042"  Part="1"
-F 0 "#PWR042" H 4850 5300 50  0001 C CNN
+AR Path="/5D766247/5F151EC9" Ref="#PWR045"  Part="1"
+F 0 "#PWR045" H 4850 5300 50  0001 C CNN
 F 1 "+5V" H 4865 5623 50  0000 C CNN
 F 2 "" H 4850 5450 50  0001 C CNN
@@
 P 2050 5250
 AR Path="/5C4C7509/5F151ED3" Ref="#PWR?"  Part="1"
-AR Path="/5D766247/5F151ED3" Ref="#PWR034"  Part="1"
-F 0 "#PWR034" H 2050 5100 50  0001 C CNN
+AR Path="/5D766247/5F151ED3" Ref="#PWR037"  Part="1"
+F 0 "#PWR037" H 2050 5100 50  0001 C CNN
 F 1 "+5V" H 2065 5423 50  0000 C CNN
 F 2 "" H 2050 5250 50  0001 C CNN
@@
 VT: Voltage/Temperature\nI: Current (Amperes)
 $Comp
-L Connector_Generic:Conn_01x04 J6
+L Connector_Generic:Conn_01x04 J7
 U 1 1 5F1F64D7
 P 9400 4200
-F 0 "J6" H 9480 4192 50  0000 L CNN
+F 0 "J7" H 9480 4192 50  0000 L CNN
 F 1 "CurrentConn" H 9480 4101 50  0000 L CNN
-F 2 "" H 9400 4200 50  0001 C CNN
+F 2 "Connector_Molex:Molex_Micro-Fit_3.0_43650-0415_1x04_P3.00mm_Vertical" H 9400 4200 50  0001 C CNN
 F 3 "~" H 9400 4200 50  0001 C CNN
 	1    9400 4200
@@
 $EndComp
 $Comp
-L power:+12V #PWR046
+L power:+12V #PWR049
 U 1 1 5F1F84DF
 P 9100 4000
-F 0 "#PWR046" H 9100 3850 50  0001 C CNN
+F 0 "#PWR049" H 9100 3850 50  0001 C CNN
 F 1 "+12V" H 9115 4173 50  0000 C CNN
 F 2 "" H 9100 4000 50  0001 C CNN
@@
 $EndComp
 $Comp
-L power:GNDPWR #PWR047
+L power:GNDPWR #PWR050
 U 1 1 5F1F8DBA
 P 9100 4500
-F 0 "#PWR047" H 9100 4300 50  0001 C CNN
+F 0 "#PWR050" H 9100 4300 50  0001 C CNN
 F 1 "GNDPWR" H 9104 4346 50  0000 C CNN
 F 2 "" H 9100 4450 50  0001 C CNN
@@
 Wire Wire Line
 	9100 4400 9100 4500
-Text Notes 8800 3000 0    100  ~ 20
+Text Notes 8950 3000 0    100  ~ 20
 Connectors
 Wire Wire Line
