File: BPS/FanBoard/FanBoard/FanBoard.sch (KiCad schematic (older format))
At the start: 8 parts, among them J1 Conn_01x02, J2 Conn_01x02, J3 Conn_01x02, J4 Conn_01x02

Commit message: Finished schematic for Fan Board:)
Parts:
- added D1, D2, D3, D4: C3D25170H, Package_TO_SOT_THT:TO-247-2_Vertical, symbol Diode:C3D25170H
- gave numbers to parts that had none: 4
Connections:
- wire segments 13 -> 29
Other:
- moved on the sheet: J1, J2, J3, J4
Changed lines of the file:
@@
 L Connector_Generic:Conn_01x02 J1
 U 1 1 5F091D5D
-P 4250 3750
-F 0 "J1" H 4330 3742 50  0000 L CNN
-F 1 "Conn_01x02" H 4330 3651 50  0000 L CNN
-F 2 "" H 4250 3750 50  0001 C CNN
-F 3 "~" H 4250 3750 50  0001 C CNN
-	1    4250 3750
+P 4250 3650
+F 0 "J1" H 4330 3642 50  0000 L CNN
+F 1 "Conn_01x02" H 4330 3551 50  0000 L CNN
+F 2 "" H 4250 3650 50  0001 C CNN
+F 3 "~" H 4250 3650 50  0001 C CNN
+	1    4250 3650
 	1    0    0    -1
 $EndComp
@@
 L Connector_Generic:Conn_01x02 J2
 U 1 1 5F09203F
-P 4250 4400
-F 0 "J2" H 4330 4392 50  0000 L CNN
-F 1 "Conn_01x02" H 4330 4301 50  0000 L CNN
-F 2 "" H 4250 4400 50  0001 C CNN
-F 3 "~" H 4250 4400 50  0001 C CNN
-	1    4250 4400
+P 4250 4300
+F 0 "J2" H 4330 4292 50  0000 L CNN
+F 1 "Conn_01x02" H 4330 4201 50  0000 L CNN
+F 2 "" H 4250 4300 50  0001 C CNN
+F 3 "~" H 4250 4300 50  0001 C CNN
+	1    4250 4300
 	1    0    0    -1
 $EndComp
@@
 L Connector_Generic:Conn_01x02 J3
 U 1 1 5F092588
-P 4250 5050
-F 0 "J3" H 4330 5042 50  0000 L CNN
-F 1 "Conn_01x02" H 4330 4951 50  0000 L CNN
-F 2 "" H 4250 5050 50  0001 C CNN
-F 3 "~" H 4250 5050 50  0001 C CNN
-	1    4250 5050
+P 4250 4950
+F 0 "J3" H 4330 4942 50  0000 L CNN
+F 1 "Conn_01x02" H 4330 4851 50  0000 L CNN
+F 2 "" H 4250 4950 50  0001 C CNN
+F 3 "~" H 4250 4950 50  0001 C CNN
+	1    4250 4950
 	1    0    0    -1
 $EndComp
@@
 L Connector_Generic:Conn_01x02 J4
 U 1 1 5F092946
-P 4250 5700
-F 0 "J4" H 4330 5692 50  0000 L CNN
-F 1 "Conn_01x02" H 4330 5601 50  0000 L CNN
-F 2 "" H 4250 5700 50  0001 C CNN
-F 3 "~" H 4250 5700 50  0001 C CNN
-	1    4250 5700
+P 4250 5600
+F 0 "J4" H 4330 5592 50  0000 L CNN
+F 1 "Conn_01x02" H 4330 5501 50  0000 L CNN
+F 2 "" H 4250 5600 50  0001 C CNN
+F 3 "~" H 4250 5600 50  0001 C CNN
+	1    4250 5600
 	1    0    0    -1
 $EndComp
@@
 L power:+12V #PWR01
 U 1 1 5F093D32
-P 3950 3600
-F 0 "#PWR01" H 3950 3450 50  0001 C CNN
-F 1 "+12V" H 3965 3773 50  0000 C CNN
-F 2 "" H 3950 3600 50  0001 C CNN
-F 3 "" H 3950 3600 50  0001 C CNN
-	1    3950 3600
-	1    0    0    -1
-$EndComp
-Wire Wire Line
-	3200 4400 4050 4400
+P 3550 3450
+F 0 "#PWR01" H 3550 3300 50  0001 C CNN
+F 1 "+12V" H 3565 3623 50  0000 C CNN
+F 2 "" H 3550 3450 50  0001 C CNN
+F 3 "" H 3550 3450 50  0001 C CNN
+	1    3550 3450
+	1    0    0    -1
+$EndComp
+Wire Wire Line
+	3200 4400 3700 4400
 Wire Wire Line
 	3200 5050 4050 5050
@@
 NoConn ~ 2900 4600
 NoConn ~ 2900 3950
-Connection ~ 4050 5700
-Wire Wire Line
-	4050 5700 4100 5700
-$Comp
-L Transistor_FET:BUK9M34-100EX Q?
+$Comp
+L Transistor_FET:BUK9M34-100EX Q1
 U 1 1 5F0AEA0D
 P 3100 3950
-F 0 "Q?" H 3304 3996 50  0000 L CNN
+F 0 "Q1" H 3304 3996 50  0000 L CNN
 F 1 "BUK9M34-100EX" H 3304 3905 50  0000 L CNN
 F 2 "Package_TO_SOT_SMD:LFPAK33" H 3300 3875 50  0001 L CIN
@@
 $EndComp
 $Comp
-L Transistor_FET:BUK9M34-100EX Q?
+L Transistor_FET:BUK9M34-100EX Q2
 U 1 1 5F0B1145
 P 3100 4600
-F 0 "Q?" H 3304 4646 50  0000 L CNN
+F 0 "Q2" H 3304 4646 50  0000 L CNN
 F 1 "BUK9M34-100EX" H 3304 4555 50  0000 L CNN
 F 2 "Package_TO_SOT_SMD:LFPAK33" H 3300 4525 50  0001 L CIN
@@
 $EndComp
 $Comp
-L Transistor_FET:BUK9M34-100EX Q?
+L Transistor_FET:BUK9M34-100EX Q3
 U 1 1 5F0B279A
 P 3100 5250
-F 0 "Q?" H 3304 5296 50  0000 L CNN
+F 0 "Q3" H 3304 5296 50  0000 L CNN
 F 1 "BUK9M34-100EX" H 3304 5205 50  0000 L CNN
 F 2 "Package_TO_SOT_SMD:LFPAK33" H 3300 5175 50  0001 L CIN
@@
 $EndComp
 $Comp
-L Transistor_FET:BUK9M34-100EX Q?
+L Transistor_FET:BUK9M34-100EX Q4
 U 1 1 5F0B2EF7
 P 3100 5900
-F 0 "Q?" H 3304 5946 50  0000 L CNN
+F 0 "Q4" H 3304 5946 50  0000 L CNN
 F 1 "BUK9M34-100EX" H 3304 5855 50  0000 L CNN
 F 2 "Package_TO_SOT_SMD:LFPAK33" H 3300 5825 50  0001 L CIN
@@
 $EndComp
 Wire Wire Line
-	3200 5700 4050 5700
-Wire Wire Line
 	3200 4150 3600 4150
 Wire Wire Line
@@
 	3600 4800 3600 5450
 $Comp
-L power:GND #PWR?
+L power:GND #PWR02
 U 1 1 5F0B61B4
 P 3600 6200
-F 0 "#PWR?" H 3600 5950 50  0001 C CNN
+F 0 "#PWR02" H 3600 5950 50  0001 C CNN
 F 1 "GND" H 3605 6027 50  0000 C CNN
 F 2 "" H 3600 6200 50  0001 C CNN
@@
 Wire Wire Line
 	3600 6100 3600 6200
+$Comp
+L Diode:C3D25170H D2
+U 1 1 5F0A0D46
+P 3700 4250
+F 0 "D2" V 3700 4350 50  0000 L CNN
+F 1 "C3D25170H" V 3600 4300 50  0000 L CNN
+F 2 "Package_TO_SOT_THT:TO-247-2_Vertical" H 3700 4075 50  0001 C CNN
+F 3 "https://www.wolfspeed.com/media/downloads/103/C3D25170H.pdf" H 3700 4250 50  0001 C CNN
+	1    3700 4250
+	0    1    1    0
+$EndComp
+Wire Wire Line
+	3200 5700 4050 5700
+Connection ~ 3700 4400
+Wire Wire Line
+	3700 4400 4050 4400
+$Comp
+L Diode:C3D25170H D1
+U 1 1 5F0A355E
+P 3700 3600
+F 0 "D1" V 3700 3700 50  0000 L CNN
+F 1 "C3D25170H" V 3600 3650 50  0000 L CNN
+F 2 "Package_TO_SOT_THT:TO-247-2_Vertical" H 3700 3425 50  0001 C CNN
+F 3 "https://www.wolfspeed.com/media/downloads/103/C3D25170H.pdf" H 3700 3600 50  0001 C CNN
+	1    3700 3600
+	0    1    1    0
+$EndComp
+$Comp
+L Diode:C3D25170H D3
+U 1 1 5F0A37E3
+P 3700 4900
+F 0 "D3" V 3700 5000 50  0000 L CNN
+F 1 "C3D25170H" V 3600 4950 50  0000 L CNN
+F 2 "Package_TO_SOT_THT:TO-247-2_Vertical" H 3700 4725 50  0001 C CNN
+F 3 "https://www.wolfspeed.com/media/downloads/103/C3D25170H.pdf" H 3700 4900 50  0001 C CNN
+	1    3700 4900
+	0    1    1    0
+$EndComp
+$Comp
+L Diode:C3D25170H D4
+U 1 1 5F0A3942
+P 3750 5550
+F 0 "D4" V 3750 5650 50  0000 L CNN
+F 1 "C3D25170H" V 3650 5600 50  0000 L CNN
+F 2 "Package_TO_SOT_THT:TO-247-2_Vertical" H 3750 5375 50  0001 C CNN
+F 3 "https://www.wolfspeed.com/media/downloads/103/C3D25170H.pdf" H 3750 5550 50  0001 C CNN
+	1    3750 5550
+	0    1    1    0
+$EndComp
+Wire Wire Line
+	4050 5600 3950 5600
+Wire Wire Line
+	3950 5600 3950 5400
+Wire Wire Line
+	3950 3450 3700 3450
+Connection ~ 3700 3450
+Wire Wire Line
+	3700 3450 3550 3450
+Wire Wire Line
+	4050 3650 3950 3650
+Connection ~ 3950 3650
+Wire Wire Line
+	3950 3650 3950 3450
+Wire Wire Line
+	3950 4100 3700 4100
+Connection ~ 3950 4100
+Wire Wire Line
+	3950 4100 3950 3650
+Wire Wire Line
+	4050 4300 3950 4300
+Connection ~ 3950 4300
+Wire Wire Line
+	3950 4300 3950 4100
+Wire Wire Line
+	3700 4750 3950 4750
+Connection ~ 3950 4750
+Wire Wire Line
+	3950 4750 3950 4300
+Wire Wire Line
+	4050 4950 3950 4950
+Connection ~ 3950 4950
+Wire Wire Line
+	3950 4950 3950 4750
+Wire Wire Line
+	3750 5400 3950 5400
+Connection ~ 3950 5400
+Wire Wire Line
+	3950 5400 3950 4950
 $EndSCHEMATC
